Commit message: Update table collision meshes

File: assets/environment/table_description/urdf/table.urdf (copy).xacro (robot description, xacro)
@@ -5,10 +5,10 @@
 	  <visual name="None">
 	    <geometry>
-	      <mesh filename="package://table_description/meshes/visual/table.stl" scale="0.001000 0.001000 0.001000"/>
+	      <mesh filename="package://table_description/meshes/collision/table.stl" scale="0.001000 0.001000 0.001000"/>
 	    </geometry>
 	  </visual>
 	  <collision name="None">
 	    <geometry>
-	      <mesh filename="package://table_description/meshes/visual/table.stl" scale="0.001000 0.001000 0.001000"/>
+	      <mesh filename="package://table_description/meshes/collision/table.stl" scale="0.001000 0.001000 0.001000"/>
 	    </geometry>
 	  </collision>

File: assets/environment/table_description/urdf/table.urdf.xacro (robot description, xacro)
@@ -5,10 +5,10 @@
 	  <visual name="table_${prefix}">
 	    <geometry>
-	      <mesh filename="package://table_description/meshes/visual/table.stl" scale="0.001000 0.001000 0.001000"/>
+	      <mesh filename="package://table_description/meshes/collision/table.stl" scale="0.001000 0.001000 0.001000"/>
 	    </geometry>
 	  </visual>
 	  <collision name="None_${prefix}">
 	    <geometry>
-	      <mesh filename="package://table_description/meshes/visual/table.stl" scale="0.001000 0.001000 0.001000"/>
+	      <mesh filename="package://table_description/meshes/collision/table.stl" scale="0.001000 0.001000 0.001000"/>
 	    </geometry>
 	  </collision>
