Commit message: Use dedicated collision mesh for table description

File: assets/environment/table_description/urdf/table.urdf.xacro (robot description, xacro)
@@ -10,5 +10,5 @@
 	  <collision name="None_${prefix}">
 	    <geometry>
-	      <mesh filename="package://table_description/meshes/visual/table.stl" scale="0.001000 0.001000 0.001000"/>
+	      <mesh filename="package://table_description/meshes/collision/table.stl" scale="0.001000 0.001000 0.001000"/>
 	    </geometry>
 	  </collision>
