Commit message: Fix universal robot xacro references

File: scenes/new_scene/urdf/scene.urdf.xacro (robot description, xacro)
@@ -2,8 +2,11 @@
 <robot xmlns:xacro="http://www.ros.org/wiki/xacro" name="new_scene">
  <link name="world"/>
- <xacro:include filename="$(find ur_description)/urdf/ur.urdf.xacro"/>
- <xacro:ur_robot name="ur5" tf_prefix="" parent="world" joint_limits_parameters_file="$(find ur_description)/config/ur5/joint_limits.yaml" kinematics_parameters_file="$(find ur_description)/config/ur5/default_kinematics.yaml" physical_parameters_file="$(find ur_description)/config/ur5/physical_parameters.yaml" visual_parameters_file="$(find ur_description)/config/ur5/visual_parameters.yaml" safety_limits="false" safety_pos_margin="0.15" safety_k_position="20" force_abs_paths="false">
+ <xacro:include filename="$(find ur_description)/urdf/ur5.urdf.xacro"/>
+ <xacro:ur5_robot prefix="" joint_limited="false"/>
+  <joint name="world_ur5" type="fixed">
+	<parent link="world" />
+	<child link="base_link" />
 	<origin xyz="0 0 0" rpy="0 0 0"/>
- </xacro:ur_robot>
+  </joint>
  <xacro:include filename="$(find robotiq_85_description)/urdf/robotiq_85_gripper.urdf.xacro"/>
  <xacro:robotiq_85_gripper prefix="" parent="tool0">
