Commit message: Add UR description legacy check in fixture xacro

File: assets/end_effectors/single_suction_gripper/single_suction_description/urdf/ur5_double_fixture.urdf.xacro (robot description, xacro)
@@ -2,19 +2,38 @@
 <robot xmlns:xacro="http://ros.org/wiki/xacro"
        name="ur5_double_fixture" >
+<xacro:arg name="ur_type" default="ur5"/>
+<xacro:arg name="name" default="ur5"/>
+<xacro:arg name="tf_prefix" default="ur5"/>
 <xacro:arg name="limited" default="true"/>
+<xacro:property name="legacy_urdf_exists" value="$(eval xacro.isfile('$(find ur_description)/urdf/$(arg ur_type).urdf.xacro'))"/>
 <!-- LOAD IN UR5 -->
 <link name="world"/>
-<!-- <xacro:include filename="$(find ur_description)/urdf/gazebo.urdf.xacro" /> -->
-<xacro:include filename="$(find ur_description)/urdf/ur5.urdf.xacro"/>
-<joint name="world_joint" type="fixed" >
-  <parent link="world" />
-  <child link = "base_link"/>
-  <origin xyz= "0.0 0.0 0.0" rpy="0.0 0.0 0.0" />
-</joint>
-<xacro:ur5_robot prefix="" joint_limited="true"/>
+<xacro:if value="${legacy_urdf_exists}">
+  <!-- <xacro:include filename="$(find ur_description)/urdf/gazebo.urdf.xacro" /> -->
+  <xacro:include filename="$(find ur_description)/urdf/ur5.urdf.xacro"/>
+  <joint name="world_joint" type="fixed" >
+    <parent link="world" />
+    <child link = "$(arg tf_prefix)base_link"/>
+    <origin xyz= "0.0 0.0 0.0" rpy="0.0 0.0 0.0" />
+  </joint>
+  <xacro:ur5_robot prefix="$(arg tf_prefix)" joint_limited="true"/>
+</xacro:if>
+<xacro:unless value="${legacy_urdf_exists}">
+  <xacro:include filename="$(find ur_description)/urdf/ur_macro.xacro"/>
+  <xacro:ur_robot
+    name="$(arg name)"
+    tf_prefix="$(arg tf_prefix)"
+    parent="world"
+    joint_limits_parameters_file="$(find ur_description)/config/$(arg ur_type)/joint_limits.yaml"
+    kinematics_parameters_file="$(find ur_description)/config/$(arg ur_type)/default_kinematics.yaml"
+    physical_parameters_file="$(find ur_description)/config/$(arg ur_type)/physical_parameters.yaml"
+    visual_parameters_file="$(find ur_description)/config/$(arg ur_type)/visual_parameters.yaml">
+    <origin xyz="0 0 0" rpy="0 0 0"/>
+  </xacro:ur_robot>
+</xacro:unless>
 <!-- Robotiq Gripper -->
 <xacro:include filename="$(find dual_gripper)/urdf/double_end_effector.urdf.xacro"/>
 <joint name="ur5_to_double_fixture" type="fixed">
-	<parent link="tool0" />
+	<parent link="$(arg tf_prefix)tool0" />
 	<child link="ref"/>
 	<origin xyz= "0 0 0" rpy="${-pi/2} ${pi} ${3*pi/2}"/>

Commit message: Update UR5 xacros for ur_description v2

File: assets/end_effectors/single_suction_gripper/single_suction_description/urdf/ur5_double_fixture.urdf.xacro (robot description, xacro)
@@ -6,30 +6,19 @@
 <xacro:arg name="tf_prefix" default="ur5"/>
 <xacro:arg name="limited" default="true"/>
-<xacro:property name="legacy_urdf_exists" value="$(eval xacro.isfile('$(find ur_description)/urdf/$(arg ur_type).urdf.xacro'))"/>
 <!-- LOAD IN UR5 -->
 <link name="world"/>
-<xacro:if value="${legacy_urdf_exists}">
-  <!-- <xacro:include filename="$(find ur_description)/urdf/gazebo.urdf.xacro" /> -->
-  <xacro:include filename="$(find ur_description)/urdf/ur5.urdf.xacro"/>
-  <joint name="world_joint" type="fixed" >
-    <parent link="world" />
-    <child link = "$(arg tf_prefix)base_link"/>
-    <origin xyz= "0.0 0.0 0.0" rpy="0.0 0.0 0.0" />
-  </joint>
-  <xacro:ur5_robot prefix="$(arg tf_prefix)" joint_limited="true"/>
-</xacro:if>
-<xacro:unless value="${legacy_urdf_exists}">
-  <xacro:include filename="$(find ur_description)/urdf/ur_macro.xacro"/>
-  <xacro:ur_robot
-    name="$(arg name)"
-    tf_prefix="$(arg tf_prefix)"
-    parent="world"
-    joint_limits_parameters_file="$(find ur_description)/config/$(arg ur_type)/joint_limits.yaml"
-    kinematics_parameters_file="$(find ur_description)/config/$(arg ur_type)/default_kinematics.yaml"
-    physical_parameters_file="$(find ur_description)/config/$(arg ur_type)/physical_parameters.yaml"
-    visual_parameters_file="$(find ur_description)/config/$(arg ur_type)/visual_parameters.yaml">
-    <origin xyz="0 0 0" rpy="0 0 0"/>
-  </xacro:ur_robot>
-</xacro:unless>
+<xacro:include filename="$(find ur_description)/urdf/ur_macro.xacro"/>
+<xacro:ur_robot
+  name="$(arg name)"
+  tf_prefix="$(arg tf_prefix)"
+  joint_limit_params="$(find ur_description)/config/$(arg ur_type)/joint_limits.yaml"
+  kinematics_params="$(find ur_description)/config/$(arg ur_type)/default_kinematics.yaml"
+  physical_params="$(find ur_description)/config/$(arg ur_type)/physical_parameters.yaml"
+  visual_params="$(find ur_description)/config/$(arg ur_type)/visual_parameters.yaml"/>
+<joint name="world_joint" type="fixed" >
+  <parent link="world" />
+  <child link = "$(arg tf_prefix)base_link"/>
+  <origin xyz= "0.0 0.0 0.0" rpy="0.0 0.0 0.0" />
+</joint>
 <!-- Robotiq Gripper -->
 <xacro:include filename="$(find dual_gripper)/urdf/double_end_effector.urdf.xacro"/>

File: scenes/suction_test/urdf/scene.urdf.xacro (robot description, xacro)
@@ -4,15 +4,13 @@
  <xacro:arg name="name" default="$(arg ur_type)"/>
  <xacro:arg name="tf_prefix" default=""/>
- <xacro:property name="legacy_ur_xacro" value="$(find ur_description)/urdf/$(arg ur_type).urdf.xacro"/>
- <xacro:property name="legacy_ur_available" value="$(eval xacro.file_exists(legacy_ur_xacro))"/>
  <link name="world"/>
- <xacro:if value="${legacy_ur_available}">
-  <xacro:include filename="$(find ur_description)/urdf/ur5.urdf.xacro"/>
-  <xacro:ur5_robot prefix="" joint_limited="false"/>
- </xacro:if>
- <xacro:unless value="${legacy_ur_available}">
-  <xacro:include filename="$(find ur_description)/urdf/ur_macro.xacro"/>
-  <xacro:ur_robot name="$(arg name)" tf_prefix="$(arg tf_prefix)" joint_limit_params="$(find ur_description)/config/$(arg ur_type)/joint_limits.yaml" kinematics_params="$(find ur_description)/config/$(arg ur_type)/default_kinematics.yaml" physical_params="$(find ur_description)/config/$(arg ur_type)/physical_parameters.yaml" visual_params="$(find ur_description)/config/$(arg ur_type)/visual_parameters.yaml"/>
- </xacro:unless>
+ <xacro:include filename="$(find ur_description)/urdf/ur_macro.xacro"/>
+ <xacro:ur_robot
+  name="$(arg name)"
+  tf_prefix="$(arg tf_prefix)"
+  joint_limit_params="$(find ur_description)/config/$(arg ur_type)/joint_limits.yaml"
+  kinematics_params="$(find ur_description)/config/$(arg ur_type)/default_kinematics.yaml"
+  physical_params="$(find ur_description)/config/$(arg ur_type)/physical_parameters.yaml"
+  visual_params="$(find ur_description)/config/$(arg ur_type)/visual_parameters.yaml"/>
   <joint name="world_ur5" type="fixed">
 	<parent link="world" />
@@ -38,10 +36,9 @@
     <origin xyz="-0.58 0.225 0.65" rpy="3.14159 1.57079506 0"/>
 </xacro:sensor_d415>
-<link name="ee_palm" />​
-​
-<joint name="base_to_palm" type="fixed">​
-    <parent link="suction_cup_link"/>​
-    <child link="ee_palm"/>​
-    <origin xyz="0 0 0" rpy="-3.14159 0 1.57079506"/>​
+<link name="ee_palm" />
+<joint name="base_to_palm" type="fixed">
+    <parent link="suction_cup_link"/>
+    <child link="ee_palm"/>
+    <origin xyz="0 0 0" rpy="-3.14159 0 1.57079506"/>
 </joint>
 </robot>

File: scenes/ur5_2f_test/urdf/scene.urdf.xacro (robot description, xacro)
@@ -4,15 +4,13 @@
  <xacro:arg name="name" default="$(arg ur_type)"/>
  <xacro:arg name="tf_prefix" default=""/>
- <xacro:property name="legacy_ur_xacro" value="$(find ur_description)/urdf/$(arg ur_type).urdf.xacro"/>
- <xacro:property name="legacy_ur_available" value="$(eval xacro.file_exists(legacy_ur_xacro))"/>
  <link name="world"/>
- <xacro:if value="${legacy_ur_available}">
-  <xacro:include filename="$(find ur_description)/urdf/ur5.urdf.xacro"/>
-  <xacro:ur5_robot prefix="" joint_limited="false"/>
- </xacro:if>
- <xacro:unless value="${legacy_ur_available}">
-  <xacro:include filename="$(find ur_description)/urdf/ur_macro.xacro"/>
-  <xacro:ur_robot name="$(arg name)" tf_prefix="$(arg tf_prefix)" joint_limit_params="$(find ur_description)/config/$(arg ur_type)/joint_limits.yaml" kinematics_params="$(find ur_description)/config/$(arg ur_type)/default_kinematics.yaml" physical_params="$(find ur_description)/config/$(arg ur_type)/physical_parameters.yaml" visual_params="$(find ur_description)/config/$(arg ur_type)/visual_parameters.yaml"/>
- </xacro:unless>
+ <xacro:include filename="$(find ur_description)/urdf/ur_macro.xacro"/>
+ <xacro:ur_robot
+  name="$(arg name)"
+  tf_prefix="$(arg tf_prefix)"
+  joint_limit_params="$(find ur_description)/config/$(arg ur_type)/joint_limits.yaml"
+  kinematics_params="$(find ur_description)/config/$(arg ur_type)/default_kinematics.yaml"
+  physical_params="$(find ur_description)/config/$(arg ur_type)/physical_parameters.yaml"
+  visual_params="$(find ur_description)/config/$(arg ur_type)/visual_parameters.yaml"/>
   <joint name="world_ur5" type="fixed">
 	<parent link="world" />

File: scenes/ur5_3f_test/urdf/scene.urdf.xacro (robot description, xacro)
@@ -4,15 +4,13 @@
  <xacro:arg name="name" default="$(arg ur_type)"/>
  <xacro:arg name="tf_prefix" default=""/>
- <xacro:property name="legacy_ur_xacro" value="$(find ur_description)/urdf/$(arg ur_type).urdf.xacro"/>
- <xacro:property name="legacy_ur_available" value="$(eval xacro.file_exists(legacy_ur_xacro))"/>
  <link name="world"/>
- <xacro:if value="${legacy_ur_available}">
-  <xacro:include filename="$(find ur_description)/urdf/ur5.urdf.xacro"/>
-  <xacro:ur5_robot prefix="" joint_limited="false"/>
- </xacro:if>
- <xacro:unless value="${legacy_ur_available}">
-  <xacro:include filename="$(find ur_description)/urdf/ur_macro.xacro"/>
-  <xacro:ur_robot name="$(arg name)" tf_prefix="$(arg tf_prefix)" joint_limit_params="$(find ur_description)/config/$(arg ur_type)/joint_limits.yaml" kinematics_params="$(find ur_description)/config/$(arg ur_type)/default_kinematics.yaml" physical_params="$(find ur_description)/config/$(arg ur_type)/physical_parameters.yaml" visual_params="$(find ur_description)/config/$(arg ur_type)/visual_parameters.yaml"/>
- </xacro:unless>
+ <xacro:include filename="$(find ur_description)/urdf/ur_macro.xacro"/>
+ <xacro:ur_robot
+  name="$(arg name)"
+  tf_prefix="$(arg tf_prefix)"
+  joint_limit_params="$(find ur_description)/config/$(arg ur_type)/joint_limits.yaml"
+  kinematics_params="$(find ur_description)/config/$(arg ur_type)/default_kinematics.yaml"
+  physical_params="$(find ur_description)/config/$(arg ur_type)/physical_parameters.yaml"
+  visual_params="$(find ur_description)/config/$(arg ur_type)/visual_parameters.yaml"/>
   <joint name="world_ur5" type="fixed">
 	<parent link="world" />

File: scenes/ur5_airpick4_test/urdf/scene.urdf.xacro (robot description, xacro)
@@ -4,15 +4,13 @@
  <xacro:arg name="name" default="$(arg ur_type)"/>
  <xacro:arg name="tf_prefix" default=""/>
- <xacro:property name="legacy_ur_xacro" value="$(find ur_description)/urdf/$(arg ur_type).urdf.xacro"/>
- <xacro:property name="legacy_ur_available" value="$(eval xacro.file_exists(legacy_ur_xacro))"/>
  <link name="world"/>
- <xacro:if value="${legacy_ur_available}">
-  <xacro:include filename="$(find ur_description)/urdf/ur5.urdf.xacro"/>
-  <xacro:ur5_robot prefix="" joint_limited="false"/>
- </xacro:if>
- <xacro:unless value="${legacy_ur_available}">
-  <xacro:include filename="$(find ur_description)/urdf/ur_macro.xacro"/>
-  <xacro:ur_robot name="$(arg name)" tf_prefix="$(arg tf_prefix)" joint_limit_params="$(find ur_description)/config/$(arg ur_type)/joint_limits.yaml" kinematics_params="$(find ur_description)/config/$(arg ur_type)/default_kinematics.yaml" physical_params="$(find ur_description)/config/$(arg ur_type)/physical_parameters.yaml" visual_params="$(find ur_description)/config/$(arg ur_type)/visual_parameters.yaml"/>
- </xacro:unless>
+ <xacro:include filename="$(find ur_description)/urdf/ur_macro.xacro"/>
+ <xacro:ur_robot
+  name="$(arg name)"
+  tf_prefix="$(arg tf_prefix)"
+  joint_limit_params="$(find ur_description)/config/$(arg ur_type)/joint_limits.yaml"
+  kinematics_params="$(find ur_description)/config/$(arg ur_type)/default_kinematics.yaml"
+  physical_params="$(find ur_description)/config/$(arg ur_type)/physical_parameters.yaml"
+  visual_params="$(find ur_description)/config/$(arg ur_type)/visual_parameters.yaml"/>
   <joint name="world_ur5" type="fixed">
 	<parent link="world" />

Commit message: Attach UR robots to world

File: assets/end_effectors/single_suction_gripper/single_suction_description/urdf/ur5_double_fixture.urdf.xacro (robot description, xacro)
@@ -12,13 +12,11 @@
   name="$(arg name)"
   tf_prefix="$(arg tf_prefix)"
+  parent="world"
   joint_limits_parameters_file="$(find ur_description)/config/$(arg ur_type)/joint_limits.yaml"
   kinematics_params="$(find ur_description)/config/$(arg ur_type)/default_kinematics.yaml"
   physical_params="$(find ur_description)/config/$(arg ur_type)/physical_parameters.yaml"
-  visual_params="$(find ur_description)/config/$(arg ur_type)/visual_parameters.yaml"/>
-<joint name="world_joint" type="fixed" >
-  <parent link="world" />
-  <child link = "$(arg tf_prefix)base_link"/>
-  <origin xyz= "0.0 0.0 0.0" rpy="0.0 0.0 0.0" />
-</joint>
+  visual_params="$(find ur_description)/config/$(arg ur_type)/visual_parameters.yaml">
+  <origin xyz="0 0 0" rpy="0 0 0"/>
+</xacro:ur_robot>
 <!-- Robotiq Gripper -->
 <xacro:include filename="$(find dual_gripper)/urdf/double_end_effector.urdf.xacro"/>

File: scenes/suction_test/urdf/scene.urdf.xacro (robot description, xacro)
@@ -9,8 +9,11 @@
   name="$(arg name)"
   tf_prefix="$(arg tf_prefix)"
+  parent="world"
   joint_limits_parameters_file="$(find ur_description)/config/$(arg ur_type)/joint_limits.yaml"
   kinematics_params="$(find ur_description)/config/$(arg ur_type)/default_kinematics.yaml"
   physical_params="$(find ur_description)/config/$(arg ur_type)/physical_parameters.yaml"
-  visual_params="$(find ur_description)/config/$(arg ur_type)/visual_parameters.yaml"/>
+  visual_params="$(find ur_description)/config/$(arg ur_type)/visual_parameters.yaml">
+  <origin xyz="0 0 0" rpy="0 0 0"/>
+</xacro:ur_robot>
  <!-- Import ur5 ros2_control description -->
 <xacro:include filename="$(find ur5_moveit_config)/config/ur5.ros2_control.xacro" />

File: scenes/ur5_2f_test/urdf/scene.urdf.xacro (robot description, xacro)
@@ -9,8 +9,11 @@
   name="$(arg name)"
   tf_prefix="$(arg tf_prefix)"
+  parent="world"
   joint_limits_parameters_file="$(find ur_description)/config/$(arg ur_type)/joint_limits.yaml"
   kinematics_params="$(find ur_description)/config/$(arg ur_type)/default_kinematics.yaml"
   physical_params="$(find ur_description)/config/$(arg ur_type)/physical_parameters.yaml"
-  visual_params="$(find ur_description)/config/$(arg ur_type)/visual_parameters.yaml"/>
+  visual_params="$(find ur_description)/config/$(arg ur_type)/visual_parameters.yaml">
+  <origin xyz="0 0 0" rpy="0 0 0"/>
+ </xacro:ur_robot>
  <!-- Import ur5 ros2_control description -->
  <xacro:include filename="$(find ur5_moveit_config)/config/ur5.ros2_control.xacro" />

File: scenes/ur5_3f_test/urdf/scene.urdf.xacro (robot description, xacro)
@@ -9,8 +9,11 @@
   name="$(arg name)"
   tf_prefix="$(arg tf_prefix)"
+  parent="world"
   joint_limits_parameters_file="$(find ur_description)/config/$(arg ur_type)/joint_limits.yaml"
   kinematics_params="$(find ur_description)/config/$(arg ur_type)/default_kinematics.yaml"
   physical_params="$(find ur_description)/config/$(arg ur_type)/physical_parameters.yaml"
-  visual_params="$(find ur_description)/config/$(arg ur_type)/visual_parameters.yaml"/>
+  visual_params="$(find ur_description)/config/$(arg ur_type)/visual_parameters.yaml">
+  <origin xyz="0 0 0" rpy="0 0 0"/>
+ </xacro:ur_robot>
  <!-- Import ur5 ros2_control description -->
  <xacro:include filename="$(find ur5_moveit_config)/config/ur5.ros2_control.xacro" />

File: scenes/ur5_airpick4_test/urdf/scene.urdf.xacro (robot description, xacro)
@@ -9,8 +9,11 @@
   name="$(arg name)"
   tf_prefix="$(arg tf_prefix)"
+  parent="world"
   joint_limits_parameters_file="$(find ur_description)/config/$(arg ur_type)/joint_limits.yaml"
   kinematics_params="$(find ur_description)/config/$(arg ur_type)/default_kinematics.yaml"
   physical_params="$(find ur_description)/config/$(arg ur_type)/physical_parameters.yaml"
-  visual_params="$(find ur_description)/config/$(arg ur_type)/visual_parameters.yaml"/>
+  visual_params="$(find ur_description)/config/$(arg ur_type)/visual_parameters.yaml">
+  <origin xyz="0 0 0" rpy="0 0 0"/>
+ </xacro:ur_robot>
  <!-- Import ur5 ros2_control description -->
  <xacro:include filename="$(find ur5_moveit_config)/config/ur5.ros2_control.xacro" />
