Commit message: Render complete suction end effector

File: assets/end_effectors/single_suction_gripper/single_suction_description/urdf/single_suction_gripper.urdf.xacro (robot description, xacro)
@@ -38,5 +38,19 @@
       </link>
       <link name="suction_cup_link">
-        <origin xyz= "-0.22836 0.053 0"/>
+        <visual>
+          <origin xyz="0 0 0" rpy="0 0 0" />
+          <geometry>
+            <mesh filename="package://single_suction_description/meshes/suction_cup_link.STL" />
+          </geometry>
+          <material name="">
+            <color rgba="0.15 0.15 0.15 1" />
+          </material>
+        </visual>
+        <collision>
+          <origin xyz="0 0 0" rpy="0 0 0" />
+          <geometry>
+            <mesh filename="package://single_suction_description/meshes/suction_cup_link.STL" />
+          </geometry>
+        </collision>
       </link>
       <joint name="virtual_ee_joint" type="fixed">

File: scenes/suction_test/urdf/scene.urdf.xacro (robot description, xacro)
@@ -10,5 +10,5 @@
  <xacro:arg name="camera_world_xyz" default=""/>
  <xacro:arg name="camera_world_rpy" default=""/>
- <xacro:arg name="suction_mount_rpy" default="-1.5708 -1.5708 0"/>
+ <xacro:arg name="suction_mount_rpy" default="1.5707 -1.5707 0"/>
  <link name="$(arg world_frame)"/>
 <xacro:include filename="$(find ur_description)/urdf/ur_macro.xacro"/>
@@ -27,5 +27,4 @@
 <xacro:include filename="$(find single_suction_description)/urdf/single_suction_gripper.urdf.xacro"/>
 <xacro:single_suction_gripper prefix="" parent="tool0">
- <!-- virtual_ee_joint rotates cup +Z onto fixture +X; this mount maps it to world -Z at preview home. -->
  <origin xyz="0 0 0" rpy="$(arg suction_mount_rpy)"/>
  </xacro:single_suction_gripper>
