Commit message: Replace ee_link with tool0 in UR SRDFs

File: assets/robots/universal_robot/ur10_moveit_config/config/ur10.srdf.xacro (robot description, xacro)
@@ -12,8 +12,8 @@
     <!--SUBGROUPS: Groups can also be formed by referencing to already defined group names-->
     <group name="manipulator">
-        <chain base_link="base_link" tip_link="ee_link"/>
+        <chain base_link="base_link" tip_link="tool0"/>
     </group>
     <group name="endeffector">
-        <link name="ee_link"/>
+        <link name="tool0"/>
     </group>
     <!--GROUP STATES: Purpose: Define a named state for a particular group, in terms of joint values. This is useful to define states like 'folded arms'-->
@@ -35,5 +35,5 @@
     </group_state>
     <!--END EFFECTOR: Purpose: Represent information about an end effector.-->
-    <end_effector name="moveit_ee" parent_link="ee_link" group="endeffector" />
+    <end_effector name="moveit_ee" parent_link="tool0" group="endeffector" />
     <!--VIRTUAL JOINT: Purpose: this element defines a virtual joint between a robot link and an external frame of reference (considered fixed with respect to the robot)-->
     <virtual_joint name="fixed_base" type="fixed" parent_frame="world" child_link="base_link" />
@@ -42,7 +42,7 @@
     <disable_collisions link1="base_link" link2="upper_arm_link" reason="Never" />
     <disable_collisions link1="base_link" link2="wrist_1_link" reason="Never" />
-    <disable_collisions link1="ee_link" link2="wrist_1_link" reason="Never" />
-    <disable_collisions link1="ee_link" link2="wrist_2_link" reason="Never" />
-    <disable_collisions link1="ee_link" link2="wrist_3_link" reason="Adjacent" />
+    <disable_collisions link1="tool0" link2="wrist_1_link" reason="Never" />
+    <disable_collisions link1="tool0" link2="wrist_2_link" reason="Never" />
+    <disable_collisions link1="tool0" link2="wrist_3_link" reason="Adjacent" />
     <disable_collisions link1="forearm_link" link2="upper_arm_link" reason="Adjacent" />
     <disable_collisions link1="forearm_link" link2="wrist_1_link" reason="Adjacent" />

File: assets/robots/universal_robot/ur3_moveit_config/config/ur3.srdf.xacro (robot description, xacro)
@@ -12,8 +12,8 @@
     <!--SUBGROUPS: Groups can also be formed by referencing to already defined group names-->
     <group name="manipulator">
-        <chain base_link="base_link" tip_link="ee_link" />
+        <chain base_link="base_link" tip_link="tool0" />
     </group>
     <group name="endeffector">
-        <link name="ee_link" />
+        <link name="tool0" />
     </group>
     <!--GROUP STATES: Purpose: Define a named state for a particular group, in terms of joint values. This is useful to define states like 'folded arms'-->
@@ -35,12 +35,12 @@
     </group_state>
     <!--END EFFECTOR: Purpose: Represent information about an end effector.-->
-    <end_effector name="moveit_ee" parent_link="ee_link" group="endeffector" />
+    <end_effector name="moveit_ee" parent_link="tool0" group="endeffector" />
     <!--VIRTUAL JOINT: Purpose: this element defines a virtual joint between a robot link and an external frame of reference (considered fixed with respect to the robot)-->
     <virtual_joint name="fixed_base" type="fixed" parent_frame="world" child_link="base_link" />
     <!--DISABLE COLLISIONS: By default it is assumed that any link of the robot could potentially come into collision with any other link in the robot. This tag disables collision checking between a specified pair of links. -->
     <disable_collisions link1="base_link" link2="shoulder_link" reason="Adjacent" />
-    <disable_collisions link1="ee_link" link2="wrist_1_link" reason="Never" />
-    <disable_collisions link1="ee_link" link2="wrist_2_link" reason="Never" />
-    <disable_collisions link1="ee_link" link2="wrist_3_link" reason="Adjacent" />
+    <disable_collisions link1="tool0" link2="wrist_1_link" reason="Never" />
+    <disable_collisions link1="tool0" link2="wrist_2_link" reason="Never" />
+    <disable_collisions link1="tool0" link2="wrist_3_link" reason="Adjacent" />
     <disable_collisions link1="forearm_link" link2="upper_arm_link" reason="Adjacent" />
     <disable_collisions link1="forearm_link" link2="wrist_1_link" reason="Adjacent" />

File: assets/robots/universal_robot/ur5_moveit_config/config/ur5.srdf.xacro (robot description, xacro)
@@ -12,8 +12,8 @@
     <!--SUBGROUPS: Groups can also be formed by referencing to already defined group names-->
     <group name="manipulator">
-        <chain base_link="base_link" tip_link="ee_link" />
+        <chain base_link="base_link" tip_link="tool0" />
     </group>
     <group name="endeffector">
-        <link name="ee_link" />
+        <link name="tool0" />
     </group>
     <!--GROUP STATES: Purpose: Define a named state for a particular group, in terms of joint values. This is useful to define states like 'folded arms'-->
@@ -35,12 +35,12 @@
     </group_state>
     <!--END EFFECTOR: Purpose: Represent information about an end effector.-->
-    <end_effector name="moveit_ee" parent_link="ee_link" group="endeffector" />
+    <end_effector name="moveit_ee" parent_link="tool0" group="endeffector" />
     <!--VIRTUAL JOINT: Purpose: this element defines a virtual joint between a robot link and an external frame of reference (considered fixed with respect to the robot)-->
     <virtual_joint name="fixed_base" type="fixed" parent_frame="world" child_link="base_link" />
     <!--DISABLE COLLISIONS: By default it is assumed that any link of the robot could potentially come into collision with any other link in the robot. This tag disables collision checking between a specified pair of links. -->
     <disable_collisions link1="base_link" link2="shoulder_link" reason="Adjacent" />
-    <disable_collisions link1="ee_link" link2="wrist_1_link" reason="Never" />
-    <disable_collisions link1="ee_link" link2="wrist_2_link" reason="Never" />
-    <disable_collisions link1="ee_link" link2="wrist_3_link" reason="Adjacent" />
+    <disable_collisions link1="tool0" link2="wrist_1_link" reason="Never" />
+    <disable_collisions link1="tool0" link2="wrist_2_link" reason="Never" />
+    <disable_collisions link1="tool0" link2="wrist_3_link" reason="Adjacent" />
     <disable_collisions link1="forearm_link" link2="upper_arm_link" reason="Adjacent" />
     <disable_collisions link1="forearm_link" link2="wrist_1_link" reason="Adjacent" />
