Commit message: Add parent group to 3F gripper SRDF

File: assets/end_effectors/robotiq_3f_gripper/robotiq_3f_moveit_config/config/robotiq_3f_gripper.srdf.xacro (robot description, xacro)
@@ -5,5 +5,5 @@
 -->
 <robot xmlns:xacro="http://www.ros.org/wiki/xacro" name="robotiq-3f-gripper_articulated">
-<xacro:macro name="robotiq-3f-gripper_articulated">
+<xacro:macro name="robotiq-3f-gripper_articulated" params="parent_group:=manipulator">
     <!--GROUPS: Representation of a set of joints and links. This can be useful for specifying DOF to plan for, defining arms, end effectors, etc-->
     <!--LINKS: When a link is specified, the parent joint of that link (if it exists) is automatically included-->
@@ -27,5 +27,5 @@
         <joint name="palm_finger_middle_joint" />
     </group>
-    <end_effector name="robotiq_3f_gripper" parent_link="palm" group="gripper" />
+    <end_effector name="robotiq_3f_gripper" parent_link="palm" group="gripper" parent_group="${parent_group}" />
     <!--VIRTUAL JOINT: Purpose: this element defines a virtual joint between a robot link and an external frame of reference (considered fixed with respect to the robot)-->
     <virtual_joint name="world_joint" type="fixed" parent_frame="world" child_link="palm" />
