Commit message: Replace ee_link with tool0 in scenes and gripper

File: assets/end_effectors/robotiq_85_gripper/robotiq_85_description/urdf/kinova_robotiq_85_gripper.xacro (robot description, xacro)
@@ -40,9 +40,9 @@
     <joint name="ee_fixed_joint" type="fixed">
         <parent link="gripper_root_link" />
-        <child link = "ee_link" />
+        <child link = "tool0" />
         <origin xyz="0.202757 0 0.85" rpy="0 0 0"/>
     </joint>
-    <link name="ee_link"/>
-    <xacro:robotiq_85_kinova_coupler prefix="" parent="ee_link">
+    <link name="tool0"/>
+    <xacro:robotiq_85_kinova_coupler prefix="" parent="tool0">
         <origin xyz="-0.152757 0 0" rpy="0 ${-pi/2} 0"/>
     </xacro:robotiq_85_kinova_coupler>

File: scenes/ur5_airpick4_test/urdf/arm_hand.srdf.xacro (robot description, xacro)
@@ -12,5 +12,5 @@
   <disable_collisions link1="gripper_base_link" link2="wrist_2_link" reason="Never" />
   <disable_collisions link1="gripper_base_link" link2="wrist_3_link" reason="Never" />
-  <disable_collisions link1="gripper_base_link" link2="ee_link" reason="Never" />
+  <disable_collisions link1="gripper_base_link" link2="tool0" reason="Never" />
   <disable_collisions link1="gripper_base_link" link2="base" reason="Never" />
   <disable_collisions link1="gripper_base_link" link2="tool0" reason="Never" />
