Commit message: Fix robotiq knuckle inertials for stable RViz parsing

File: assets/end_effectors/robotiq_85_gripper/robotiq_85_description/urdf/robotiq_85_gripper.urdf.xacro (robot description, xacro)
@@ -62,8 +62,8 @@
             <inertial>
                 <mass value="0.018491" />
-                <origin xyz="0.0 0.0 0.0" />
-                <inertia ixx = "0.000009" ixy = "-0.000001" ixz = "0.000000"
-                         iyx = "-0.000001" iyy = "0.000001" iyz = "0.000000"
-                         izx = "0.000000" izy = "0.000000" izz = "0.000010" />
+                <origin xyz="0.000926 -0.017947 0.0" />
+                <inertia ixx = "0.000006" ixy = "0.000000" ixz = "0.000000"
+                         iyx = "0.000000" iyy = "0.000003" iyz = "0.000000"
+                         izx = "0.000000" izy = "0.000000" izz = "0.000006" />
             </inertial>
         </link>
@@ -88,8 +88,8 @@
             <inertial>
                 <mass value="0.018491" />
-                <origin xyz="0.0 0.0 0.0" />
-                <inertia ixx = "0.000009" ixy = "-0.000001" ixz = "0.000000"
-                         iyx = "-0.000001" iyy = "0.000001" iyz = "0.000000"
-                         izx = "0.000000" izy = "0.000000" izz = "0.000010" />
+                <origin xyz="0.000926 -0.017947 0.0" />
+                <inertia ixx = "0.000006" ixy = "0.000000" ixz = "0.000000"
+                         iyx = "0.000000" iyy = "0.000003" iyz = "0.000000"
+                         izx = "0.000000" izy = "0.000000" izz = "0.000006" />
             </inertial>
         </link>
