Commit message: Fix scene and gripper configs

File: assets/end_effectors/robotiq_85_gripper/robotiq_85_moveit_config/config/robotiq_85_gripper.srdf.xacro (robot description, xacro)
@@ -12,5 +12,4 @@
     <!--SUBGROUPS: Groups can also be formed by referencing to already defined group names-->
     <group name="gripper">
-        <joint name="kinova_robotiq_coupler_joint" />
         <joint name="gripper_base_joint" />
         <joint name="gripper_finger1_inner_knuckle_joint" />
@@ -24,5 +23,4 @@
     </group>
     <!--VIRTUAL JOINT: Purpose: this element defines a virtual joint between a robot link and an external frame of reference (considered fixed with respect to the robot)-->
-    <!--virtual_joint name="world_joint" type="fixed" parent_frame="world" child_link="gripper_root_link" /-->
     <!--PASSIVE JOINT: Purpose: this element is used to mark joints that are not actuated-->
     <passive_joint name="gripper_finger1_inner_knuckle_joint" />
@@ -40,6 +38,4 @@
     <disable_collisions link1="gripper_base_link" link2="gripper_finger2_inner_knuckle_link" reason="Adjacent" />
     <disable_collisions link1="gripper_base_link" link2="gripper_finger2_knuckle_link" reason="Adjacent" />
-    <disable_collisions link1="gripper_base_link" link2="gripper_root_link" reason="Never" />
-    <disable_collisions link1="gripper_base_link" link2="robotiq_coupler_link" reason="Adjacent" />
     <disable_collisions link1="gripper_finger1_finger_link" link2="gripper_finger1_finger_tip_link" reason="Default" />
     <disable_collisions link1="gripper_finger1_finger_link" link2="gripper_finger1_inner_knuckle_link" reason="Never" />
@@ -49,6 +45,4 @@
     <disable_collisions link1="gripper_finger1_finger_link" link2="gripper_finger2_inner_knuckle_link" reason="Never" />
     <disable_collisions link1="gripper_finger1_finger_link" link2="gripper_finger2_knuckle_link" reason="Never" />
-    <disable_collisions link1="gripper_finger1_finger_link" link2="gripper_root_link" reason="Never" />
-    <disable_collisions link1="gripper_finger1_finger_link" link2="robotiq_coupler_link" reason="Never" />
     <disable_collisions link1="gripper_finger1_finger_tip_link" link2="gripper_finger1_inner_knuckle_link" reason="Adjacent" />
     <disable_collisions link1="gripper_finger1_finger_tip_link" link2="gripper_finger1_knuckle_link" reason="Never" />
@@ -56,6 +50,4 @@
     <disable_collisions link1="gripper_finger1_finger_tip_link" link2="gripper_finger2_inner_knuckle_link" reason="Never" />
     <disable_collisions link1="gripper_finger1_finger_tip_link" link2="gripper_finger2_knuckle_link" reason="Never" />
-    <disable_collisions link1="gripper_finger1_finger_tip_link" link2="gripper_root_link" reason="Never" />
-    <disable_collisions link1="gripper_finger1_finger_tip_link" link2="robotiq_coupler_link" reason="Never" />
     <disable_collisions link1="gripper_finger1_inner_knuckle_link" link2="gripper_finger1_knuckle_link" reason="Never" />
     <disable_collisions link1="gripper_finger1_inner_knuckle_link" link2="gripper_finger2_finger_link" reason="Never" />
@@ -63,27 +55,14 @@
     <disable_collisions link1="gripper_finger1_inner_knuckle_link" link2="gripper_finger2_inner_knuckle_link" reason="Never" />
     <disable_collisions link1="gripper_finger1_inner_knuckle_link" link2="gripper_finger2_knuckle_link" reason="Never" />
-    <disable_collisions link1="gripper_finger1_inner_knuckle_link" link2="gripper_root_link" reason="Never" />
-    <disable_collisions link1="gripper_finger1_inner_knuckle_link" link2="robotiq_coupler_link" reason="Never" />
     <disable_collisions link1="gripper_finger1_knuckle_link" link2="gripper_finger2_finger_link" reason="Never" />
     <disable_collisions link1="gripper_finger1_knuckle_link" link2="gripper_finger2_finger_tip_link" reason="Never" />
     <disable_collisions link1="gripper_finger1_knuckle_link" link2="gripper_finger2_inner_knuckle_link" reason="Never" />
     <disable_collisions link1="gripper_finger1_knuckle_link" link2="gripper_finger2_knuckle_link" reason="Never" />
-    <disable_collisions link1="gripper_finger1_knuckle_link" link2="gripper_root_link" reason="Never" />
-    <disable_collisions link1="gripper_finger1_knuckle_link" link2="robotiq_coupler_link" reason="Never" />
     <disable_collisions link1="gripper_finger2_finger_link" link2="gripper_finger2_finger_tip_link" reason="Default" />
     <disable_collisions link1="gripper_finger2_finger_link" link2="gripper_finger2_inner_knuckle_link" reason="Never" />
     <disable_collisions link1="gripper_finger2_finger_link" link2="gripper_finger2_knuckle_link" reason="Adjacent" />
-    <disable_collisions link1="gripper_finger2_finger_link" link2="gripper_root_link" reason="Never" />
-    <disable_collisions link1="gripper_finger2_finger_link" link2="robotiq_coupler_link" reason="Never" />
     <disable_collisions link1="gripper_finger2_finger_tip_link" link2="gripper_finger2_inner_knuckle_link" reason="Adjacent" />
     <disable_collisions link1="gripper_finger2_finger_tip_link" link2="gripper_finger2_knuckle_link" reason="Never" />
-    <disable_collisions link1="gripper_finger2_finger_tip_link" link2="gripper_root_link" reason="Never" />
-    <disable_collisions link1="gripper_finger2_finger_tip_link" link2="robotiq_coupler_link" reason="Never" />
     <disable_collisions link1="gripper_finger2_inner_knuckle_link" link2="gripper_finger2_knuckle_link" reason="Never" />
-    <disable_collisions link1="gripper_finger2_inner_knuckle_link" link2="gripper_root_link" reason="Never" />
-    <disable_collisions link1="gripper_finger2_inner_knuckle_link" link2="robotiq_coupler_link" reason="Never" />
-    <disable_collisions link1="gripper_finger2_knuckle_link" link2="gripper_root_link" reason="Never" />
-    <disable_collisions link1="gripper_finger2_knuckle_link" link2="robotiq_coupler_link" reason="Never" />
-    <disable_collisions link1="gripper_root_link" link2="robotiq_coupler_link" reason="Adjacent" />
 </xacro:macro>
 </robot>

File: assets/robots/universal_robot/ur10_moveit_config/config/ur10.ros2_control.xacro (robot description, xacro)
@@ -2,5 +2,5 @@
 <robot xmlns:xacro="http://www.ros.org/wiki/xacro">
     <xacro:macro name="ur10_ros2_control" params="name initial_positions_file">
-        <xacro:property name="initial_positions" value="${load_yaml(initial_positions_file)['initial_positions']}"/>
+        <xacro:property name="initial_positions" value="${xacro.load_yaml(initial_positions_file)['initial_positions']}"/>
         <ros2_control name="${name}" type="system">
             <hardware>

File: assets/robots/universal_robot/ur3_moveit_config/config/ur3.ros2_control.xacro (robot description, xacro)
@@ -2,5 +2,5 @@
 <robot xmlns:xacro="http://www.ros.org/wiki/xacro">
     <xacro:macro name="ur3_ros2_control" params="name initial_positions_file">
-        <xacro:property name="initial_positions" value="${load_yaml(initial_positions_file)['initial_positions']}"/>
+        <xacro:property name="initial_positions" value="${xacro.load_yaml(initial_positions_file)['initial_positions']}"/>
         <ros2_control name="${name}" type="system">
             <hardware>

File: assets/robots/universal_robot/ur5_moveit_config/config/ur5.ros2_control.xacro (robot description, xacro)
@@ -2,5 +2,5 @@
 <robot xmlns:xacro="http://www.ros.org/wiki/xacro">
     <xacro:macro name="ur5_ros2_control" params="name initial_positions_file">
-        <xacro:property name="initial_positions" value="${load_yaml(initial_positions_file)['initial_positions']}"/>
+        <xacro:property name="initial_positions" value="${xacro.load_yaml(initial_positions_file)['initial_positions']}"/>
         <ros2_control name="${name}" type="system">
             <hardware>

File: scenes/ur5_2f_test/urdf/arm_hand.srdf.xacro (robot description, xacro)
@@ -1,4 +1,4 @@
 <?xml version="1.0" ?>
-<robot xmlns:xacro="http://www.ros.org/wiki/xacro" name="ur5_test">
+<robot xmlns:xacro="http://www.ros.org/wiki/xacro" name="ur5_2f_test">
   <xacro:include filename="$(find ur5_moveit_config)/config/ur5.srdf.xacro" />
   <xacro:include filename="$(find robotiq_85_moveit_config)/config/robotiq_85_gripper.srdf.xacro" />

File: scenes/ur5_2f_test/urdf/scene.urdf.xacro (robot description, xacro)
@@ -1,4 +1,4 @@
 <?xml version="1.0" ?>
-<robot xmlns:xacro="http://www.ros.org/wiki/xacro" name="ur5_test">
+<robot xmlns:xacro="http://www.ros.org/wiki/xacro" name="ur5_2f_test">
  <link name="world"/>
  <xacro:include filename="$(find ur_description)/urdf/ur5.urdf.xacro"/>
@@ -17,5 +17,5 @@
 	<origin xyz="0 0 0" rpy="1.5707 -1.5707 0"/>
  </xacro:robotiq_85_gripper>
- <xacro:include filename="$(find workbench_description)/urdf/table.urdf.xacro"/>
+ <xacro:include filename="$(find table_description)/urdf/table.urdf.xacro"/>
  <xacro:table prefix="" parent="world">
 	<origin xyz="0 0 0" rpy="0 0 0"/>

File: scenes/ur5_3f_test/urdf/scene.urdf.xacro (robot description, xacro)
@@ -21,5 +21,5 @@
 	<origin xyz="0 0 0.0" rpy="1.5707 0 0"/>
  </xacro:robotiq-3f-gripper_articulated>
- <xacro:include filename="$(find workbench_description)/urdf/table.urdf.xacro"/>
+ <xacro:include filename="$(find table_description)/urdf/table.urdf.xacro"/>
  <xacro:table prefix="" parent="world">
 	<origin xyz="0 0 0" rpy="0 0 0"/>

File: scenes/ur5_airpick4_test/urdf/scene.urdf.xacro (robot description, xacro)
@@ -13,5 +13,5 @@
  <xacro:arg name="initial_positions_file" default="$(find ur5_moveit_config)/config/initial_positions.yaml" />
  <xacro:ur5_ros2_control name="UR5FakeSystem" initial_positions_file="$(arg initial_positions_file)"/>
- <xacro:include filename="$(find workbench_description)/urdf/table.urdf.xacro"/>
+ <xacro:include filename="$(find table_description)/urdf/table.urdf.xacro"/>
  <xacro:table prefix="" parent="world">
 	<origin xyz="0 0 0" rpy="0 0 0"/>

Commit message: Fix robotiq SRDF and update UR scene xacro

File: assets/end_effectors/robotiq_85_gripper/robotiq_85_moveit_config/config/robotiq_85_gripper.srdf.xacro (robot description, xacro)
@@ -13,5 +13,4 @@
     <group name="gripper">
         <chain base_link="gripper_base_link" tip_link="gripper_finger1_finger_tip_link" />
-        <joint name="kinova_robotiq_coupler_joint" />
         <joint name="gripper_base_joint" />
         <joint name="gripper_finger1_inner_knuckle_joint" />
@@ -24,5 +23,5 @@
         <joint name="gripper_finger2_finger_joint" />
     </group>
-    <end_effector name="robotiq_85_gripper" parent_link="tool0" group="gripper" parent_group="${parent_group}" />
+    <end_effector name="robotiq_85_gripper" parent_link="tool0" group="gripper" parent_group="manipulator" />
     <!--VIRTUAL JOINT: Purpose: this element defines a virtual joint between a robot link and an external frame of reference (considered fixed with respect to the robot)-->
     <!--virtual_joint name="world_joint" type="fixed" parent_frame="world" child_link="gripper_root_link" /-->
@@ -42,6 +41,4 @@
     <disable_collisions link1="gripper_base_link" link2="gripper_finger2_inner_knuckle_link" reason="Adjacent" />
     <disable_collisions link1="gripper_base_link" link2="gripper_finger2_knuckle_link" reason="Adjacent" />
-    <disable_collisions link1="gripper_base_link" link2="gripper_root_link" reason="Never" />
-    <disable_collisions link1="gripper_base_link" link2="robotiq_coupler_link" reason="Adjacent" />
     <disable_collisions link1="gripper_finger1_finger_link" link2="gripper_finger1_finger_tip_link" reason="Default" />
     <disable_collisions link1="gripper_finger1_finger_link" link2="gripper_finger1_inner_knuckle_link" reason="Never" />
@@ -51,6 +48,4 @@
     <disable_collisions link1="gripper_finger1_finger_link" link2="gripper_finger2_inner_knuckle_link" reason="Never" />
     <disable_collisions link1="gripper_finger1_finger_link" link2="gripper_finger2_knuckle_link" reason="Never" />
-    <disable_collisions link1="gripper_finger1_finger_link" link2="gripper_root_link" reason="Never" />
-    <disable_collisions link1="gripper_finger1_finger_link" link2="robotiq_coupler_link" reason="Never" />
     <disable_collisions link1="gripper_finger1_finger_tip_link" link2="gripper_finger1_inner_knuckle_link" reason="Adjacent" />
     <disable_collisions link1="gripper_finger1_finger_tip_link" link2="gripper_finger1_knuckle_link" reason="Never" />
@@ -58,6 +53,4 @@
     <disable_collisions link1="gripper_finger1_finger_tip_link" link2="gripper_finger2_inner_knuckle_link" reason="Never" />
     <disable_collisions link1="gripper_finger1_finger_tip_link" link2="gripper_finger2_knuckle_link" reason="Never" />
-    <disable_collisions link1="gripper_finger1_finger_tip_link" link2="gripper_root_link" reason="Never" />
-    <disable_collisions link1="gripper_finger1_finger_tip_link" link2="robotiq_coupler_link" reason="Never" />
     <disable_collisions link1="gripper_finger1_inner_knuckle_link" link2="gripper_finger1_knuckle_link" reason="Never" />
     <disable_collisions link1="gripper_finger1_inner_knuckle_link" link2="gripper_finger2_finger_link" reason="Never" />
@@ -65,27 +58,14 @@
     <disable_collisions link1="gripper_finger1_inner_knuckle_link" link2="gripper_finger2_inner_knuckle_link" reason="Never" />
     <disable_collisions link1="gripper_finger1_inner_knuckle_link" link2="gripper_finger2_knuckle_link" reason="Never" />
-    <disable_collisions link1="gripper_finger1_inner_knuckle_link" link2="gripper_root_link" reason="Never" />
-    <disable_collisions link1="gripper_finger1_inner_knuckle_link" link2="robotiq_coupler_link" reason="Never" />
     <disable_collisions link1="gripper_finger1_knuckle_link" link2="gripper_finger2_finger_link" reason="Never" />
     <disable_collisions link1="gripper_finger1_knuckle_link" link2="gripper_finger2_finger_tip_link" reason="Never" />
     <disable_collisions link1="gripper_finger1_knuckle_link" link2="gripper_finger2_inner_knuckle_link" reason="Never" />
     <disable_collisions link1="gripper_finger1_knuckle_link" link2="gripper_finger2_knuckle_link" reason="Never" />
-    <disable_collisions link1="gripper_finger1_knuckle_link" link2="gripper_root_link" reason="Never" />
-    <disable_collisions link1="gripper_finger1_knuckle_link" link2="robotiq_coupler_link" reason="Never" />
     <disable_collisions link1="gripper_finger2_finger_link" link2="gripper_finger2_finger_tip_link" reason="Default" />
     <disable_collisions link1="gripper_finger2_finger_link" link2="gripper_finger2_inner_knuckle_link" reason="Never" />
     <disable_collisions link1="gripper_finger2_finger_link" link2="gripper_finger2_knuckle_link" reason="Adjacent" />
-    <disable_collisions link1="gripper_finger2_finger_link" link2="gripper_root_link" reason="Never" />
-    <disable_collisions link1="gripper_finger2_finger_link" link2="robotiq_coupler_link" reason="Never" />
     <disable_collisions link1="gripper_finger2_finger_tip_link" link2="gripper_finger2_inner_knuckle_link" reason="Adjacent" />
     <disable_collisions link1="gripper_finger2_finger_tip_link" link2="gripper_finger2_knuckle_link" reason="Never" />
-    <disable_collisions link1="gripper_finger2_finger_tip_link" link2="gripper_root_link" reason="Never" />
-    <disable_collisions link1="gripper_finger2_finger_tip_link" link2="robotiq_coupler_link" reason="Never" />
     <disable_collisions link1="gripper_finger2_inner_knuckle_link" link2="gripper_finger2_knuckle_link" reason="Never" />
-    <disable_collisions link1="gripper_finger2_inner_knuckle_link" link2="gripper_root_link" reason="Never" />
-    <disable_collisions link1="gripper_finger2_inner_knuckle_link" link2="robotiq_coupler_link" reason="Never" />
-    <disable_collisions link1="gripper_finger2_knuckle_link" link2="gripper_root_link" reason="Never" />
-    <disable_collisions link1="gripper_finger2_knuckle_link" link2="robotiq_coupler_link" reason="Never" />
-    <disable_collisions link1="gripper_root_link" link2="robotiq_coupler_link" reason="Adjacent" />
 </xacro:macro>
 </robot>
