Commit message: Add UR xacro args with legacy fallback

File: scenes/suction_test/urdf/scene.urdf.xacro (robot description, xacro)
@@ -1,7 +1,18 @@
 <?xml version="1.0" ?>
 <robot xmlns:xacro="http://www.ros.org/wiki/xacro" name="suction_test">
+ <xacro:arg name="ur_type" default="ur5"/>
+ <xacro:arg name="name" default="$(arg ur_type)"/>
+ <xacro:arg name="tf_prefix" default=""/>
+ <xacro:property name="legacy_ur_xacro" value="$(find ur_description)/urdf/$(arg ur_type).urdf.xacro"/>
+ <xacro:property name="legacy_ur_available" value="$(eval xacro.file_exists(legacy_ur_xacro))"/>
  <link name="world"/>
- <xacro:include filename="$(find ur_description)/urdf/ur5.urdf.xacro"/>
- <xacro:ur5_robot prefix="" joint_limited="false"/>
+ <xacro:if value="${legacy_ur_available}">
+  <xacro:include filename="$(find ur_description)/urdf/ur5.urdf.xacro"/>
+  <xacro:ur5_robot prefix="" joint_limited="false"/>
+ </xacro:if>
+ <xacro:unless value="${legacy_ur_available}">
+  <xacro:include filename="$(find ur_description)/urdf/ur_macro.xacro"/>
+  <xacro:ur_robot name="$(arg name)" tf_prefix="$(arg tf_prefix)" joint_limit_params="$(find ur_description)/config/$(arg ur_type)/joint_limits.yaml" kinematics_params="$(find ur_description)/config/$(arg ur_type)/default_kinematics.yaml" physical_params="$(find ur_description)/config/$(arg ur_type)/physical_parameters.yaml" visual_params="$(find ur_description)/config/$(arg ur_type)/visual_parameters.yaml"/>
+ </xacro:unless>
   <joint name="world_ur5" type="fixed">
 	<parent link="world" />

File: scenes/ur5_2f_test/urdf/scene.urdf.xacro (robot description, xacro)
@@ -1,7 +1,18 @@
 <?xml version="1.0" ?>
 <robot xmlns:xacro="http://www.ros.org/wiki/xacro" name="ur5_test">
+ <xacro:arg name="ur_type" default="ur5"/>
+ <xacro:arg name="name" default="$(arg ur_type)"/>
+ <xacro:arg name="tf_prefix" default=""/>
+ <xacro:property name="legacy_ur_xacro" value="$(find ur_description)/urdf/$(arg ur_type).urdf.xacro"/>
+ <xacro:property name="legacy_ur_available" value="$(eval xacro.file_exists(legacy_ur_xacro))"/>
  <link name="world"/>
- <xacro:include filename="$(find ur_description)/urdf/ur5.urdf.xacro"/>
- <xacro:ur5_robot prefix="" joint_limited="false"/>
+ <xacro:if value="${legacy_ur_available}">
+  <xacro:include filename="$(find ur_description)/urdf/ur5.urdf.xacro"/>
+  <xacro:ur5_robot prefix="" joint_limited="false"/>
+ </xacro:if>
+ <xacro:unless value="${legacy_ur_available}">
+  <xacro:include filename="$(find ur_description)/urdf/ur_macro.xacro"/>
+  <xacro:ur_robot name="$(arg name)" tf_prefix="$(arg tf_prefix)" joint_limit_params="$(find ur_description)/config/$(arg ur_type)/joint_limits.yaml" kinematics_params="$(find ur_description)/config/$(arg ur_type)/default_kinematics.yaml" physical_params="$(find ur_description)/config/$(arg ur_type)/physical_parameters.yaml" visual_params="$(find ur_description)/config/$(arg ur_type)/visual_parameters.yaml"/>
+ </xacro:unless>
   <joint name="world_ur5" type="fixed">
 	<parent link="world" />

File: scenes/ur5_3f_test/urdf/scene.urdf.xacro (robot description, xacro)
@@ -1,7 +1,18 @@
 <?xml version="1.0" ?>
 <robot xmlns:xacro="http://www.ros.org/wiki/xacro" name="ur5_3f_test">
+ <xacro:arg name="ur_type" default="ur5"/>
+ <xacro:arg name="name" default="$(arg ur_type)"/>
+ <xacro:arg name="tf_prefix" default=""/>
+ <xacro:property name="legacy_ur_xacro" value="$(find ur_description)/urdf/$(arg ur_type).urdf.xacro"/>
+ <xacro:property name="legacy_ur_available" value="$(eval xacro.file_exists(legacy_ur_xacro))"/>
  <link name="world"/>
- <xacro:include filename="$(find ur_description)/urdf/ur5.urdf.xacro"/>
- <xacro:ur5_robot prefix="" joint_limited="false"/>
+ <xacro:if value="${legacy_ur_available}">
+  <xacro:include filename="$(find ur_description)/urdf/ur5.urdf.xacro"/>
+  <xacro:ur5_robot prefix="" joint_limited="false"/>
+ </xacro:if>
+ <xacro:unless value="${legacy_ur_available}">
+  <xacro:include filename="$(find ur_description)/urdf/ur_macro.xacro"/>
+  <xacro:ur_robot name="$(arg name)" tf_prefix="$(arg tf_prefix)" joint_limit_params="$(find ur_description)/config/$(arg ur_type)/joint_limits.yaml" kinematics_params="$(find ur_description)/config/$(arg ur_type)/default_kinematics.yaml" physical_params="$(find ur_description)/config/$(arg ur_type)/physical_parameters.yaml" visual_params="$(find ur_description)/config/$(arg ur_type)/visual_parameters.yaml"/>
+ </xacro:unless>
   <joint name="world_ur5" type="fixed">
 	<parent link="world" />

File: scenes/ur5_airpick4_test/urdf/scene.urdf.xacro (robot description, xacro)
@@ -1,7 +1,18 @@
 <?xml version="1.0" ?>
 <robot xmlns:xacro="http://www.ros.org/wiki/xacro" name="ur5_airpick4_test">
+ <xacro:arg name="ur_type" default="ur5"/>
+ <xacro:arg name="name" default="$(arg ur_type)"/>
+ <xacro:arg name="tf_prefix" default=""/>
+ <xacro:property name="legacy_ur_xacro" value="$(find ur_description)/urdf/$(arg ur_type).urdf.xacro"/>
+ <xacro:property name="legacy_ur_available" value="$(eval xacro.file_exists(legacy_ur_xacro))"/>
  <link name="world"/>
- <xacro:include filename="$(find ur_description)/urdf/ur5.urdf.xacro"/>
- <xacro:ur5_robot prefix="" joint_limited="false"/>
+ <xacro:if value="${legacy_ur_available}">
+  <xacro:include filename="$(find ur_description)/urdf/ur5.urdf.xacro"/>
+  <xacro:ur5_robot prefix="" joint_limited="false"/>
+ </xacro:if>
+ <xacro:unless value="${legacy_ur_available}">
+  <xacro:include filename="$(find ur_description)/urdf/ur_macro.xacro"/>
+  <xacro:ur_robot name="$(arg name)" tf_prefix="$(arg tf_prefix)" joint_limit_params="$(find ur_description)/config/$(arg ur_type)/joint_limits.yaml" kinematics_params="$(find ur_description)/config/$(arg ur_type)/default_kinematics.yaml" physical_params="$(find ur_description)/config/$(arg ur_type)/physical_parameters.yaml" visual_params="$(find ur_description)/config/$(arg ur_type)/visual_parameters.yaml"/>
+ </xacro:unless>
   <joint name="world_ur5" type="fixed">
 	<parent link="world" />

Commit message: Update ur_robot parameters in scenes

File: scenes/suction_test/urdf/scene.urdf.xacro (robot description, xacro)
@@ -6,11 +6,14 @@
  <link name="world"/>
 <xacro:include filename="$(find ur_description)/urdf/ur_macro.xacro"/>
- <xacro:ur_robot
+<xacro:ur_robot
   name="$(arg name)"
   tf_prefix="$(arg tf_prefix)"
-  joint_limit_params="$(find ur_description)/config/$(arg ur_type)/joint_limits.yaml"
-  kinematics_params="$(find ur_description)/config/$(arg ur_type)/default_kinematics.yaml"
-  physical_params="$(find ur_description)/config/$(arg ur_type)/physical_parameters.yaml"
-  visual_params="$(find ur_description)/config/$(arg ur_type)/visual_parameters.yaml"/>
+  joint_limits_parameters_file="$(find ur_description)/config/$(arg ur_type)/joint_limits.yaml"
+  kinematics_parameters_file="$(find ur_description)/config/$(arg ur_type)/default_kinematics.yaml"
+  physical_parameters_file="$(find ur_description)/config/$(arg ur_type)/physical_parameters.yaml"
+  visual_parameters_file="$(find ur_description)/config/$(arg ur_type)/visual_parameters.yaml"
+  parent="world">
+  <origin xyz="0 0 0" rpy="0 0 0"/>
+ </xacro:ur_robot>
   <joint name="world_ur5" type="fixed">
 	<parent link="world" />

File: scenes/ur5_2f_test/urdf/scene.urdf.xacro (robot description, xacro)
@@ -9,8 +9,11 @@
   name="$(arg name)"
   tf_prefix="$(arg tf_prefix)"
-  joint_limit_params="$(find ur_description)/config/$(arg ur_type)/joint_limits.yaml"
-  kinematics_params="$(find ur_description)/config/$(arg ur_type)/default_kinematics.yaml"
-  physical_params="$(find ur_description)/config/$(arg ur_type)/physical_parameters.yaml"
-  visual_params="$(find ur_description)/config/$(arg ur_type)/visual_parameters.yaml"/>
+  joint_limits_parameters_file="$(find ur_description)/config/$(arg ur_type)/joint_limits.yaml"
+  kinematics_parameters_file="$(find ur_description)/config/$(arg ur_type)/default_kinematics.yaml"
+  physical_parameters_file="$(find ur_description)/config/$(arg ur_type)/physical_parameters.yaml"
+  visual_parameters_file="$(find ur_description)/config/$(arg ur_type)/visual_parameters.yaml"
+  parent="world">
+  <origin xyz="0 0 0" rpy="0 0 0"/>
+ </xacro:ur_robot>
   <joint name="world_ur5" type="fixed">
 	<parent link="world" />

File: scenes/ur5_3f_test/urdf/scene.urdf.xacro (robot description, xacro)
@@ -9,8 +9,11 @@
   name="$(arg name)"
   tf_prefix="$(arg tf_prefix)"
-  joint_limit_params="$(find ur_description)/config/$(arg ur_type)/joint_limits.yaml"
-  kinematics_params="$(find ur_description)/config/$(arg ur_type)/default_kinematics.yaml"
-  physical_params="$(find ur_description)/config/$(arg ur_type)/physical_parameters.yaml"
-  visual_params="$(find ur_description)/config/$(arg ur_type)/visual_parameters.yaml"/>
+  joint_limits_parameters_file="$(find ur_description)/config/$(arg ur_type)/joint_limits.yaml"
+  kinematics_parameters_file="$(find ur_description)/config/$(arg ur_type)/default_kinematics.yaml"
+  physical_parameters_file="$(find ur_description)/config/$(arg ur_type)/physical_parameters.yaml"
+  visual_parameters_file="$(find ur_description)/config/$(arg ur_type)/visual_parameters.yaml"
+  parent="world">
+  <origin xyz="0 0 0" rpy="0 0 0"/>
+ </xacro:ur_robot>
   <joint name="world_ur5" type="fixed">
 	<parent link="world" />

File: scenes/ur5_airpick4_test/urdf/scene.urdf.xacro (robot description, xacro)
@@ -9,8 +9,11 @@
   name="$(arg name)"
   tf_prefix="$(arg tf_prefix)"
-  joint_limit_params="$(find ur_description)/config/$(arg ur_type)/joint_limits.yaml"
-  kinematics_params="$(find ur_description)/config/$(arg ur_type)/default_kinematics.yaml"
-  physical_params="$(find ur_description)/config/$(arg ur_type)/physical_parameters.yaml"
-  visual_params="$(find ur_description)/config/$(arg ur_type)/visual_parameters.yaml"/>
+  joint_limits_parameters_file="$(find ur_description)/config/$(arg ur_type)/joint_limits.yaml"
+  kinematics_parameters_file="$(find ur_description)/config/$(arg ur_type)/default_kinematics.yaml"
+  physical_parameters_file="$(find ur_description)/config/$(arg ur_type)/physical_parameters.yaml"
+  visual_parameters_file="$(find ur_description)/config/$(arg ur_type)/visual_parameters.yaml"
+  parent="world">
+  <origin xyz="0 0 0" rpy="0 0 0"/>
+ </xacro:ur_robot>
   <joint name="world_ur5" type="fixed">
 	<parent link="world" />

Commit message: Remove manual world_ur5 joints from scenes

File: scenes/suction_test/urdf/scene.urdf.xacro (robot description, xacro)
@@ -13,9 +13,4 @@
   physical_params="$(find ur_description)/config/$(arg ur_type)/physical_parameters.yaml"
   visual_params="$(find ur_description)/config/$(arg ur_type)/visual_parameters.yaml"/>
-  <joint name="world_ur5" type="fixed">
-	<parent link="world" />
-	<child link="base_link" />
-	<origin xyz="0 0 0" rpy="0 0 0"/>
-  </joint>
  <!-- Import ur5 ros2_control description -->
 <xacro:include filename="$(find ur5_moveit_config)/config/ur5.ros2_control.xacro" />

File: scenes/ur5_2f_test/urdf/scene.urdf.xacro (robot description, xacro)
@@ -13,9 +13,4 @@
   physical_params="$(find ur_description)/config/$(arg ur_type)/physical_parameters.yaml"
   visual_params="$(find ur_description)/config/$(arg ur_type)/visual_parameters.yaml"/>
-  <joint name="world_ur5" type="fixed">
-	<parent link="world" />
-	<child link="base_link" />
-	<origin xyz="0 0 0" rpy="0 0 0"/>
-  </joint>
  <!-- Import ur5 ros2_control description -->
  <xacro:include filename="$(find ur5_moveit_config)/config/ur5.ros2_control.xacro" />

File: scenes/ur5_3f_test/urdf/scene.urdf.xacro (robot description, xacro)
@@ -13,9 +13,4 @@
   physical_params="$(find ur_description)/config/$(arg ur_type)/physical_parameters.yaml"
   visual_params="$(find ur_description)/config/$(arg ur_type)/visual_parameters.yaml"/>
-  <joint name="world_ur5" type="fixed">
-	<parent link="world" />
-	<child link="base_link" />
-	<origin xyz="0 0 0" rpy="0 0 0"/>
-  </joint>
  <!-- Import ur5 ros2_control description -->
  <xacro:include filename="$(find ur5_moveit_config)/config/ur5.ros2_control.xacro" />

File: scenes/ur5_airpick4_test/urdf/scene.urdf.xacro (robot description, xacro)
@@ -13,9 +13,4 @@
   physical_params="$(find ur_description)/config/$(arg ur_type)/physical_parameters.yaml"
   visual_params="$(find ur_description)/config/$(arg ur_type)/visual_parameters.yaml"/>
-  <joint name="world_ur5" type="fixed">
-	<parent link="world" />
-	<child link="base_link" />
-	<origin xyz="0 0 0" rpy="0 0 0"/>
-  </joint>
  <!-- Import ur5 ros2_control description -->
  <xacro:include filename="$(find ur5_moveit_config)/config/ur5.ros2_control.xacro" />

Commit message: Use D435i camera model across all scene URDFs

File: scenes/suction_test/urdf/scene.urdf.xacro (robot description, xacro)
@@ -29,10 +29,10 @@
 	<origin xyz="0 0 0" rpy="0 0 0"/>
  </xacro:table>
-<xacro:include filename="$(find realsense2_description)/urdf/_d415.urdf.xacro"/>
+<xacro:include filename="$(find realsense2_description)/urdf/_d435i.urdf.xacro"/>
 <xacro:arg name="use_nominal_extrinsics" default="true" />
-<xacro:sensor_d415 parent="table_" use_nominal_extrinsics="$(arg use_nominal_extrinsics)">
+<xacro:sensor_d435i parent="table_" use_nominal_extrinsics="$(arg use_nominal_extrinsics)">
     <!--origin xyz="-0.5 0.2 0.46" rpy="0 1.57079506 0"/-->
     <origin xyz="-0.58 0.225 0.65" rpy="3.14159 1.57079506 0"/>
-</xacro:sensor_d415>
+</xacro:sensor_d435i>
 <link name="ee_palm" />
 <joint name="base_to_palm" type="fixed">

File: scenes/ur5_2f_test/urdf/scene.urdf.xacro (robot description, xacro)
@@ -29,11 +29,11 @@
 	<origin xyz="0 0 0" rpy="0 0 0"/>
  </xacro:table>
- <xacro:include filename="$(find realsense2_description)/urdf/_d415.urdf.xacro"/>
+ <xacro:include filename="$(find realsense2_description)/urdf/_d435i.urdf.xacro"/>
  <xacro:arg name="use_nominal_extrinsics" default="true" />
- <xacro:sensor_d415 parent="table_" use_nominal_extrinsics="$(arg use_nominal_extrinsics)">
+ <xacro:sensor_d435i parent="table_" use_nominal_extrinsics="$(arg use_nominal_extrinsics)">
     <origin xyz="-0.58 0.12 0.655" rpy="0 1.57079506 0"/>
- </xacro:sensor_d415>
+ </xacro:sensor_d435i>
  <link name="camera_frame" />
- <joint name="d415_to_camera" type="fixed">
+ <joint name="d435i_to_camera" type="fixed">
     <parent link="camera_link"/>
     <child link="camera_frame"/>

File: scenes/ur5_3f_test/urdf/scene.urdf.xacro (robot description, xacro)
@@ -33,9 +33,9 @@
 	<origin xyz="0 0 0" rpy="0 0 0"/>
  </xacro:table>
- <xacro:include filename="$(find realsense2_description)/urdf/_d415.urdf.xacro"/>
+ <xacro:include filename="$(find realsense2_description)/urdf/_d435i.urdf.xacro"/>
 <xacro:arg name="use_nominal_extrinsics" default="true" />
-<xacro:sensor_d415 parent="table_" use_nominal_extrinsics="$(arg use_nominal_extrinsics)">
+<xacro:sensor_d435i parent="table_" use_nominal_extrinsics="$(arg use_nominal_extrinsics)">
     <origin xyz="-0.58 0.225 0.65" rpy="3.14159 1.57079506 0"/>
-</xacro:sensor_d415>
+</xacro:sensor_d435i>
  <link name="ee_palm" />
  <joint name="base_to_palm" type="fixed">

File: scenes/ur5_airpick4_test/urdf/scene.urdf.xacro (robot description, xacro)
@@ -25,15 +25,15 @@
 	<origin xyz="0 0 0" rpy="0 0 0"/>
  </xacro:table>
-  <!--xacro:include filename="$(find realsense2_description)/urdf/_d415.urdf.xacro"/>
+  <!--xacro:include filename="$(find realsense2_description)/urdf/_d435i.urdf.xacro"/>
  <xacro:arg name="use_nominal_extrinsics" default="true" />
  <xacro:arg name="add_plug" default="true" />
- <xacro:sensor_d415 parent="table_" use_nominal_extrinsics="$(arg use_nominal_extrinsics)" add_plug="$(arg add_plug)">
+ <xacro:sensor_d435i parent="table_" use_nominal_extrinsics="$(arg use_nominal_extrinsics)" add_plug="$(arg add_plug)">
 	<origin xyz="-0.6385 0.2 0.60" rpy="0 1.57079506 0"/>
- </xacro:sensor_d415-->
- <xacro:include filename="$(find realsense2_description)/urdf/_d415.urdf.xacro"/>
+ </xacro:sensor_d435i-->
+ <xacro:include filename="$(find realsense2_description)/urdf/_d435i.urdf.xacro"/>
  <xacro:arg name="use_nominal_extrinsics" default="true" />
- <xacro:sensor_d415 parent="table_" use_nominal_extrinsics="$(arg use_nominal_extrinsics)">
+ <xacro:sensor_d435i parent="table_" use_nominal_extrinsics="$(arg use_nominal_extrinsics)">
 	<origin xyz="-0.58 0.225 0.65" rpy="3.14159 1.57079506 0"/>
- </xacro:sensor_d415>
+ </xacro:sensor_d435i>
  <xacro:include filename="$(find onrobot_airpick4_description)/urdf/onrobot_airpick4_gripper.urdf.xacro"/>
  <xacro:airpick_4_vacuum_gripper prefix="" parent="tool0">
