Commit message: fix: rename onrobot_airpick4 xacro macro from airpick_4_vacuum_gripper to onrobot_airpick4_gripper
Agent-Logs-Url: https://github.com/Mukaram01/Easy_Manipulator_Improved/sessions/58f6e8ff-0700-40cf-9e04-e5a828943efb

Co-authored-by: Mukaram01 <121873648+Mukaram01@users.noreply.github.com>

File: assets/end_effectors/onrobot_airpick4/onrobot_airpick4_description/urdf/onrobot_airpick4_gripper.urdf.xacro (robot description, xacro)
@@ -1,5 +1,5 @@
 <?xml version="1.0"?>
-<robot name="airpick_4_vacuum_gripper" xmlns:xacro="http://ros.org/wiki/xacro">
-    <xacro:macro name="airpick_4_vacuum_gripper" params="prefix parent *origin">
+<robot name="onrobot_airpick4_gripper" xmlns:xacro="http://ros.org/wiki/xacro">
+    <xacro:macro name="onrobot_airpick4_gripper" params="prefix parent *origin">
         <joint name="${prefix}gripper_base_joint" type="fixed">
             <parent link="${parent}"/>

File: assets/end_effectors/onrobot_airpick4/onrobot_airpick4_description/urdf/onrobot_airpick4_gripper_standalone.urdf.xacro (robot description, xacro)
@@ -1,10 +1,10 @@
 <?xml version="1.0"?>
-<robot name="airpick_4_vacuum_gripper" xmlns:xacro="http://ros.org/wiki/xacro">
+<robot name="onrobot_airpick4_gripper" xmlns:xacro="http://ros.org/wiki/xacro">
   <xacro:include filename="onrobot_airpick4_gripper.urdf.xacro"/>
   <xacro:arg name="prefix" default=""/>
   <xacro:arg name="parent" default="base_link"/>
   <link name="base_link"/>
-  <xacro:airpick_4_vacuum_gripper prefix="$(arg prefix)" parent="$(arg parent)">
+  <xacro:onrobot_airpick4_gripper prefix="$(arg prefix)" parent="$(arg parent)">
     <origin xyz="0 0 0" rpy="0 0 0"/>
-  </xacro:airpick_4_vacuum_gripper>
+  </xacro:onrobot_airpick4_gripper>
 </robot>

File: scenes/ur5_airpick4_test/urdf/scene.urdf.xacro (robot description, xacro)
@@ -40,7 +40,7 @@
  </xacro:sensor_d435i>
  <xacro:include filename="$(find onrobot_airpick4_description)/urdf/onrobot_airpick4_gripper.urdf.xacro"/>
- <xacro:airpick_4_vacuum_gripper prefix="" parent="tool0">
+ <xacro:onrobot_airpick4_gripper prefix="" parent="tool0">
 	<origin xyz="0 0 0.0324" rpy="-1.5707 0 0"/>
- </xacro:airpick_4_vacuum_gripper >
+ </xacro:onrobot_airpick4_gripper >
     <link name="ee_palm" />
  <joint name="base_to_palm" type="fixed">

File: workcell_builder/workcell_builder/assets/end_effectors/onrobot_airpick4/onrobot_airpick4_description/urdf/onrobot_airpick4_gripper.urdf.xacro (robot description, xacro)
@@ -1,15 +1,22 @@
 <?xml version="1.0"?>
-<robot xmlns:xacro="http://www.ros.org/wiki/xacro" name="onrobot_airpick4">
-  <link name="onrobot_airpick4_base_link">
-    <visual>
-      <geometry>
-        <box size="0.1 0.1 0.05"/>
-      </geometry>
-    </visual>
-    <collision>
-      <geometry>
-        <box size="0.1 0.1 0.05"/>
-      </geometry>
-    </collision>
-  </link>
+<robot name="onrobot_airpick4_gripper" xmlns:xacro="http://ros.org/wiki/xacro">
+    <xacro:macro name="onrobot_airpick4_gripper" params="prefix parent *origin">
+        <joint name="${prefix}gripper_base_joint" type="fixed">
+            <parent link="${parent}"/>
+            <child link="${prefix}gripper_base_link"/>
+            <xacro:insert_block name="origin"/>
+        </joint>
+       <link name="${prefix}gripper_base_link">
+            <visual>
+                <geometry>
+                    <mesh filename="package://onrobot_airpick4_description/meshes/airpick4.stl" scale="0.001000 0.001000 0.001000"/>
+                </geometry>
+            </visual>
+            <!--collision>
+                <geometry>
+                    <mesh filename="package://onrobot_airpick4_description/meshes/airpick4.stl" scale="0.001000 0.001000 0.001000"/>
+                </geometry>
+            </collision-->
+        </link>
+</xacro:macro>
 </robot>
