Commit message: fix: correct indentation in workcell_builder onrobot_airpick4 xacro
Agent-Logs-Url: https://github.com/Mukaram01/Easy_Manipulator_Improved/sessions/58f6e8ff-0700-40cf-9e04-e5a828943efb

Co-authored-by: Mukaram01 <121873648+Mukaram01@users.noreply.github.com>

File: workcell_builder/workcell_builder/assets/end_effectors/onrobot_airpick4/onrobot_airpick4_description/urdf/onrobot_airpick4_gripper.urdf.xacro (robot description, xacro)
@@ -7,5 +7,5 @@
             <xacro:insert_block name="origin"/>
         </joint>
-       <link name="${prefix}gripper_base_link">
+        <link name="${prefix}gripper_base_link">
             <visual>
                 <geometry>
