Commit message: Add end effector tags for gripper SRDFs

File: assets/end_effectors/onrobot_airpick4/onrobot_airpick4_moveit_config/config/onrobot_airpick4_gripper.srdf.xacro (robot description, xacro)
@@ -11,4 +11,8 @@
     <!--CHAINS: When a chain is specified, all the links along the chain (including endpoints) are included in the group. Additionally, all the joints that are parents to included links are also included. This means that joints along the chain and the parent joint of the base link are included in the group-->
     <!--SUBGROUPS: Groups can also be formed by referencing to already defined group names-->
+    <group name="gripper">
+        <link name="gripper_base_link" />
+    </group>
+    <end_effector name="onrobot_airpick4" parent_link="gripper_base_link" group="gripper" />
     <!--VIRTUAL JOINT: Purpose: this element defines a virtual joint between a robot link and an external frame of reference (considered fixed with respect to the robot)-->
     <virtual_joint name="world_joint" type="fixed" parent_frame="world" child_link="gripper_base_link" />

File: assets/end_effectors/robotiq_3f_gripper/robotiq_3f_moveit_config/config/robotiq_3f_gripper.srdf.xacro (robot description, xacro)
@@ -11,5 +11,6 @@
     <!--CHAINS: When a chain is specified, all the links along the chain (including endpoints) are included in the group. Additionally, all the joints that are parents to included links are also included. This means that joints along the chain and the parent joint of the base link are included in the group-->
     <!--SUBGROUPS: Groups can also be formed by referencing to already defined group names-->
-    <!--group name="gripper">
+    <group name="gripper">
+        <chain base_link="palm" tip_link="tool0" />
         <joint name="gripper_base_joint" />
         <joint name="finger_1_joint_1" />
@@ -25,5 +26,6 @@
         <joint name="palm_finger_2_joint" />
         <joint name="palm_finger_middle_joint" />
-    </group-->
+    </group>
+    <end_effector name="robotiq_3f_gripper" parent_link="palm" group="gripper" />
     <!--VIRTUAL JOINT: Purpose: this element defines a virtual joint between a robot link and an external frame of reference (considered fixed with respect to the robot)-->
     <virtual_joint name="world_joint" type="fixed" parent_frame="world" child_link="palm" />

File: assets/end_effectors/robotiq_85_gripper/robotiq_85_moveit_config/config/robotiq_85_gripper.srdf.xacro (robot description, xacro)
@@ -12,4 +12,5 @@
     <!--SUBGROUPS: Groups can also be formed by referencing to already defined group names-->
     <group name="gripper">
+        <chain base_link="gripper_base_link" tip_link="gripper_finger1_finger_tip_link" />
         <joint name="kinova_robotiq_coupler_joint" />
         <joint name="gripper_base_joint" />
@@ -23,4 +24,5 @@
         <joint name="gripper_finger2_finger_joint" />
     </group>
+    <end_effector name="robotiq_85_gripper" parent_link="gripper_base_link" group="gripper" />
     <!--VIRTUAL JOINT: Purpose: this element defines a virtual joint between a robot link and an external frame of reference (considered fixed with respect to the robot)-->
     <!--virtual_joint name="world_joint" type="fixed" parent_frame="world" child_link="gripper_root_link" /-->

File: assets/end_effectors/single_suction_gripper/single_suction_moveit_config/config/single_suction_gripper.srdf.xacro (robot description, xacro)
@@ -12,6 +12,8 @@
     <!--SUBGROUPS: Groups can also be formed by referencing to already defined group names-->
     <group name="gripper">
+        <chain base_link="wrist_fixture" tip_link="suction_cup_link" />
         <joint name="virtual_ee_joint" />
     </group>
+    <end_effector name="single_suction_gripper" parent_link="wrist_fixture" group="gripper" />
     <!--VIRTUAL JOINT: Purpose: this element defines a virtual joint between a robot link and an external frame of reference (considered fixed with respect to the robot)-->
     <!--virtual_joint name="world_joint" type="fixed" parent_frame="world" child_link="gripper_root_link" /-->

Commit message: Add parent group/link to end effector SRDFs

File: assets/end_effectors/onrobot_airpick4/onrobot_airpick4_moveit_config/config/onrobot_airpick4_gripper.srdf.xacro (robot description, xacro)
@@ -5,5 +5,5 @@
 -->
 <robot xmlns:xacro="http://www.ros.org/wiki/xacro" name="robotiq-3f-gripper_articulated">
-<xacro:macro name="onrobot_airpick4">
+<xacro:macro name="onrobot_airpick4" params="parent_group:=manipulator">
     <!--GROUPS: Representation of a set of joints and links. This can be useful for specifying DOF to plan for, defining arms, end effectors, etc-->
     <!--LINKS: When a link is specified, the parent joint of that link (if it exists) is automatically included-->
@@ -14,5 +14,5 @@
         <link name="gripper_base_link" />
     </group>
-    <end_effector name="onrobot_airpick4" parent_link="gripper_base_link" group="gripper" />
+    <end_effector name="onrobot_airpick4" parent_link="tool0" group="gripper" parent_group="${parent_group}" />
     <!--VIRTUAL JOINT: Purpose: this element defines a virtual joint between a robot link and an external frame of reference (considered fixed with respect to the robot)-->
     <virtual_joint name="world_joint" type="fixed" parent_frame="world" child_link="gripper_base_link" />

File: assets/end_effectors/robotiq_3f_gripper/robotiq_3f_moveit_config/config/robotiq_3f_gripper.srdf.xacro (robot description, xacro)
@@ -27,5 +27,5 @@
         <joint name="palm_finger_middle_joint" />
     </group>
-    <end_effector name="robotiq_3f_gripper" parent_link="palm" group="gripper" parent_group="${parent_group}" />
+    <end_effector name="robotiq_3f_gripper" parent_link="tool0" group="gripper" parent_group="${parent_group}" />
     <!--VIRTUAL JOINT: Purpose: this element defines a virtual joint between a robot link and an external frame of reference (considered fixed with respect to the robot)-->
     <virtual_joint name="world_joint" type="fixed" parent_frame="world" child_link="palm" />

File: assets/end_effectors/robotiq_85_gripper/robotiq_85_moveit_config/config/robotiq_85_gripper.srdf.xacro (robot description, xacro)
@@ -5,5 +5,5 @@
 -->
 <robot xmlns:xacro="http://www.ros.org/wiki/xacro" name="robotiq_85_gripper">
-<xacro:macro name="robotiq_85_gripper">
+<xacro:macro name="robotiq_85_gripper" params="parent_group:=manipulator">
     <!--GROUPS: Representation of a set of joints and links. This can be useful for specifying DOF to plan for, defining arms, end effectors, etc-->
     <!--LINKS: When a link is specified, the parent joint of that link (if it exists) is automatically included-->
@@ -24,5 +24,5 @@
         <joint name="gripper_finger2_finger_joint" />
     </group>
-    <end_effector name="robotiq_85_gripper" parent_link="gripper_base_link" group="gripper" />
+    <end_effector name="robotiq_85_gripper" parent_link="tool0" group="gripper" parent_group="${parent_group}" />
     <!--VIRTUAL JOINT: Purpose: this element defines a virtual joint between a robot link and an external frame of reference (considered fixed with respect to the robot)-->
     <!--virtual_joint name="world_joint" type="fixed" parent_frame="world" child_link="gripper_root_link" /-->

File: assets/robots/universal_robot/ur10_moveit_config/config/ur10.srdf.xacro (robot description, xacro)
@@ -35,5 +35,5 @@
     </group_state>
     <!--END EFFECTOR: Purpose: Represent information about an end effector.-->
-    <end_effector name="moveit_ee" parent_link="tool0" group="endeffector" />
+    <end_effector name="moveit_ee" parent_link="tool0" group="endeffector" parent_group="manipulator" />
     <!--VIRTUAL JOINT: Purpose: this element defines a virtual joint between a robot link and an external frame of reference (considered fixed with respect to the robot)-->
     <virtual_joint name="fixed_base" type="fixed" parent_frame="world" child_link="base_link" />

File: assets/robots/universal_robot/ur3_moveit_config/config/ur3.srdf.xacro (robot description, xacro)
@@ -35,5 +35,5 @@
     </group_state>
     <!--END EFFECTOR: Purpose: Represent information about an end effector.-->
-    <end_effector name="moveit_ee" parent_link="tool0" group="endeffector" />
+    <end_effector name="moveit_ee" parent_link="tool0" group="endeffector" parent_group="manipulator" />
     <!--VIRTUAL JOINT: Purpose: this element defines a virtual joint between a robot link and an external frame of reference (considered fixed with respect to the robot)-->
     <virtual_joint name="fixed_base" type="fixed" parent_frame="world" child_link="base_link" />

File: assets/robots/universal_robot/ur5_moveit_config/config/ur5.srdf.xacro (robot description, xacro)
@@ -35,5 +35,5 @@
     </group_state>
     <!--END EFFECTOR: Purpose: Represent information about an end effector.-->
-    <end_effector name="moveit_ee" parent_link="tool0" group="endeffector" />
+    <end_effector name="moveit_ee" parent_link="tool0" group="endeffector" parent_group="manipulator" />
     <!--VIRTUAL JOINT: Purpose: this element defines a virtual joint between a robot link and an external frame of reference (considered fixed with respect to the robot)-->
     <virtual_joint name="fixed_base" type="fixed" parent_frame="world" child_link="base_link" />

Commit message: Fix AirPick4 SRDF macro name for generated scenes

File: assets/end_effectors/onrobot_airpick4/onrobot_airpick4_moveit_config/config/onrobot_airpick4_gripper.srdf.xacro (robot description, xacro)
@@ -5,5 +5,5 @@
 -->
 <robot xmlns:xacro="http://www.ros.org/wiki/xacro" name="robotiq-3f-gripper_articulated">
-<xacro:macro name="onrobot_airpick4" params="parent_group:=manipulator">
+<xacro:macro name="onrobot_airpick4_gripper" params="parent_group:=manipulator">
     <!--GROUPS: Representation of a set of joints and links. This can be useful for specifying DOF to plan for, defining arms, end effectors, etc-->
     <!--LINKS: When a link is specified, the parent joint of that link (if it exists) is automatically included-->
@@ -20,3 +20,6 @@
     <!--DISABLE COLLISIONS: By default it is assumed that any link of the robot could potentially come into collision with any other link in the robot. This tag disables collision checking between a specified pair of links. -->
 </xacro:macro>
+<xacro:macro name="onrobot_airpick4" params="parent_group:=manipulator">
+    <xacro:onrobot_airpick4_gripper parent_group="${parent_group}" />
+</xacro:macro>
 </robot>
