Commit message: Fix palm inertial placement in Robotiq 3F URDF

File: assets/end_effectors/robotiq_3f_gripper/robotiq_3f_gripper_description/urdf/robotiq-3f-gripper_articulated.urdf.xacro (robot description, xacro)
@@ -374,10 +374,10 @@
       </material>
     </collision>
-  </link>
-  <inertial>
-    <origin rpy="0 0 0" xyz="0 0 0"/>
-    <mass value="1.3"/>
-    <inertia ixx="0.006012" ixy="0.000079" ixz="-0.00024" iyy="0.012892" iyz="0" izz="0.002435"/>
-  </inertial>
+    <inertial>
+      <origin rpy="0 0 0" xyz="0 0 0"/>
+      <mass value="1.3"/>
+      <inertia ixx="0.006012" ixy="0.000079" ixz="-0.00024" iyy="0.012892" iyz="0" izz="0.002435"/>
+    </inertial>
+  </link>
   <joint name="palm_finger_1_joint" type="revolute">
     <parent link="palm"/>

File: workcell_builder/workcell_builder/assets/end_effectors/robotiq_3f_gripper/robotiq_3f_gripper_description/urdf/robotiq-3f-gripper_articulated.urdf.xacro (robot description, xacro)
@@ -2,5 +2,11 @@
 <robot xmlns:xacro="http://www.ros.org/wiki/xacro" name="robotiq_3f_gripper">
   <xacro:macro name="robotiq-3f-gripper_articulated" params="prefix parent *origin">
-    <link name="${prefix}palm" />
+    <link name="${prefix}palm">
+      <inertial>
+        <origin rpy="0 0 0" xyz="0 0 0" />
+        <mass value="1.3" />
+        <inertia ixx="0.006012" ixy="0.000079" ixz="-0.00024" iyy="0.012892" iyz="0" izz="0.002435" />
+      </inertial>
+    </link>
     <joint name="${prefix}palm_joint" type="fixed">
       <parent link="${parent}" />

Commit message: fix: correct unrealistic inertia values in Robotiq 3F gripper finger and palm links
Agent-Logs-Url: https://github.com/Mukaram01/Easy_Manipulator_Improved/sessions/2ab3261f-6798-4815-84a1-7af5ab22cce5

Co-authored-by: Mukaram01 <121873648+Mukaram01@users.noreply.github.com>

File: assets/end_effectors/robotiq_3f_gripper/robotiq_3f_gripper_description/urdf/robotiq-3f-gripper_articulated.urdf.xacro (robot description, xacro)
@@ -37,5 +37,5 @@
       <origin rpy="0 0 0" xyz="0 0 0"/>
       <mass value="0.05"/>
-      <inertia ixx="0.01" ixy="-0.00002" ixz="0.00001" iyy="0.0008" iyz="0" izz="0.001"/>
+      <inertia ixx="0.001" ixy="-0.00002" ixz="0.00001" iyy="0.0008" iyz="0" izz="0.001"/>
     </inertial>
   </link>
@@ -58,5 +58,5 @@
       <origin rpy="0 0 0" xyz="0 0 0"/>
       <mass value="0.15"/>
-      <inertia ixx="0.001859" ixy="-0.000376" ixz="0.000028" iyy="0.012756" iyz="0" izz="0.0024"/>
+      <inertia ixx="0.001859" ixy="-0.000376" ixz="0.000028" iyy="0.003" iyz="0" izz="0.0024"/>
     </inertial>
   </link>
@@ -84,5 +84,5 @@
       <origin rpy="0 0 0" xyz="0 0 0"/>
       <mass value="0.15"/>
-      <inertia ixx="0.001859" ixy="-0.000376" ixz="0.000028" iyy="0.012756" iyz="0" izz="0.0024"/>
+      <inertia ixx="0.001859" ixy="-0.000376" ixz="0.000028" iyy="0.003" iyz="0" izz="0.0024"/>
     </inertial>
   </link>
@@ -151,5 +151,5 @@
       <origin rpy="0 0 0" xyz="0 0 0"/>
       <mass value="0.05"/>
-      <inertia ixx="0.01" ixy="-0.00002" ixz="0.00001" iyy="0.0008" iyz="0" izz="0.001"/>
+      <inertia ixx="0.001" ixy="-0.00002" ixz="0.00001" iyy="0.0008" iyz="0" izz="0.001"/>
     </inertial>
   </link>
@@ -172,5 +172,5 @@
       <origin rpy="0 0 0" xyz="0 0 0"/>
       <mass value="0.15"/>
-      <inertia ixx="0.001859" ixy="-0.000376" ixz="0.000028" iyy="0.012756" iyz="0" izz="0.0024"/>
+      <inertia ixx="0.001859" ixy="-0.000376" ixz="0.000028" iyy="0.003" iyz="0" izz="0.0024"/>
     </inertial>
   </link>
@@ -198,5 +198,5 @@
       <origin rpy="0 0 0" xyz="0 0 0"/>
       <mass value="0.15"/>
-      <inertia ixx="0.001859" ixy="-0.000376" ixz="0.000028" iyy="0.012756" iyz="0" izz="0.0024"/>
+      <inertia ixx="0.001859" ixy="-0.000376" ixz="0.000028" iyy="0.003" iyz="0" izz="0.0024"/>
     </inertial>
   </link>
@@ -265,5 +265,5 @@
       <origin rpy="0 0 0" xyz="0 0 0"/>
       <mass value="0.05"/>
-      <inertia ixx="0.01" ixy="-0.00002" ixz="0.00001" iyy="0.0008" iyz="0" izz="0.001"/>
+      <inertia ixx="0.001" ixy="-0.00002" ixz="0.00001" iyy="0.0008" iyz="0" izz="0.001"/>
     </inertial>
   </link>
@@ -286,5 +286,5 @@
       <origin rpy="0 0 0" xyz="0 0 0"/>
       <mass value="0.15"/>
-      <inertia ixx="0.001859" ixy="-0.000376" ixz="0.000028" iyy="0.012756" iyz="0" izz="0.0024"/>
+      <inertia ixx="0.001859" ixy="-0.000376" ixz="0.000028" iyy="0.003" iyz="0" izz="0.0024"/>
     </inertial>
   </link>
@@ -312,5 +312,5 @@
       <origin rpy="0 0 0" xyz="0 0 0"/>
       <mass value="0.15"/>
-      <inertia ixx="0.001859" ixy="-0.000376" ixz="0.000028" iyy="0.012756" iyz="0" izz="0.0024"/>
+      <inertia ixx="0.001859" ixy="-0.000376" ixz="0.000028" iyy="0.003" iyz="0" izz="0.0024"/>
     </inertial>
   </link>
@@ -377,5 +377,5 @@
       <origin rpy="0 0 0" xyz="0 0 0"/>
       <mass value="1.3"/>
-      <inertia ixx="0.006012" ixy="0.000079" ixz="-0.00024" iyy="0.012892" iyz="0" izz="0.002435"/>
+      <inertia ixx="0.006012" ixy="0.000079" ixz="-0.00024" iyy="0.008" iyz="0" izz="0.002435"/>
     </inertial>
   </link>

File: assets/end_effectors/robotiq_3f_gripper/robotiq_3f_gripper_description/urdf/robotiq-3f-gripper_articulated_macro.xacro (robot description, xacro)
@@ -34,5 +34,5 @@
             <origin xyz="0 0 0" rpy="0 0 0"/>
             <mass value="1.3"/>
-            <inertia ixx="0.006012" ixy="0.000079" ixz="-0.00024" iyy="0.012892" iyz="0" izz="0.002435" />
+            <inertia ixx="0.006012" ixy="0.000079" ixz="-0.00024" iyy="0.008" iyz="0" izz="0.002435" />
         </inertial>
 		<!-- end of link list -->

File: assets/end_effectors/robotiq_3f_gripper/robotiq_3f_gripper_description/urdf/robotiq-3f-gripper_finger_articulated_macro.xacro (robot description, xacro)
@@ -30,5 +30,5 @@
                 <origin xyz="0 0 0" rpy="0 0 0"/>
                 <mass value="0.05"/>
-                <inertia ixx="0.01" ixy="-0.00002" ixz="0.00001" iyy="0.0008" iyz="0" izz="0.001" />
+                <inertia ixx="0.001" ixy="-0.00002" ixz="0.00001" iyy="0.0008" iyz="0" izz="0.001" />
             </inertial>
 		</link>
@@ -51,5 +51,5 @@
                 <origin xyz="0 0 0" rpy="0 0 0"/>
                 <mass value="0.15"/>
-                <inertia ixx="0.001859" ixy="-0.000376" ixz="0.000028" iyy="0.012756" iyz="0" izz="0.0024" />
+                <inertia ixx="0.001859" ixy="-0.000376" ixz="0.000028" iyy="0.003" iyz="0" izz="0.0024" />
             </inertial>
 		</link>
@@ -77,5 +77,5 @@
                 <origin xyz="0 0 0" rpy="0 0 0"/>
                 <mass value="0.15"/>
-                <inertia ixx="0.001859" ixy="-0.000376" ixz="0.000028" iyy="0.012756" iyz="0" izz="0.0024" />
+                <inertia ixx="0.001859" ixy="-0.000376" ixz="0.000028" iyy="0.003" iyz="0" izz="0.0024" />
             </inertial>
 		</link>
