Commit message: Asset Library: inventory, remove stub meshes, fix inside-out models
The Builder's Asset Library is a recursive crawl of the asset roots. It
listed 103 entries, many of them single-triangle stubs drawn as distorted
triangles and six different camera mounts sharing one generic box.

- scripts/audit_asset_library.py: headless inventory reproducing the
  library crawl; per-mesh geometry, units, winding, materials, references
  and provenance. Report: docs/acceptance/asset-library-inventory-v1.
- REMOVE: 48 single-triangle stub STLs and the empty imported demo asset
  (unreferenced by scenes, URDF/xacro, generated configs or evidence).
- FIX: Robotiq 3F GRIPPER_CLOSED / GRIPPER_OPEN_FINGER_2 and the curated
  pallet.obj were inside-out (rewound); Robotiq 3F URIs pointed at the
  non-existent robotiq_3f_gripper_visualization package.
- REPLACE: packages can withhold themselves with
  <workcell_asset_library status="replace" reason="..."/>; applied to the
  six placeholder camera mounts and the empty simple_conveyor model.
- Library: unpackaged mesh + xacro are one entry; the builder-internal root
  contributes only its curated environment primitives. 103 -> 29 entries.

Co-Authored-By: Claude Opus 5.5 <noreply@anthropic.com>

File: assets/end_effectors/robotiq_3f_gripper/robotiq_3f_gripper_description/urdf/robotiq-3f-gripper_articulated.urdf (robot description, URDF)
Before this commit: robot robotiq-3f-gripper_articulated, 13 links, 12 joints
Links:
- link finger_1_link_0: geometry collision mesh filename=package://robotiq_3f_gripper_description/meshes/robotiq-3f-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; visual mesh filename=package://robotiq_3f_gripper_description/meshes/robotiq-3f-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
- link finger_1_link_1: geometry collision mesh filename=package://robotiq_3f_gripper_description/meshes/robotiq-3f-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; visual mesh filename=package://robotiq_3f_gripper_description/meshes/robotiq-3f-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
- link finger_1_link_2: geometry collision mesh filename=package://robotiq_3f_gripper_description/meshes/robotiq-3f-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; visual mesh filename=package://robotiq_3f_gripper_description/meshes/robotiq-3f-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
- link finger_1_link_3: geometry collision mesh filename=package://robotiq_3f_gripper_description/meshes/robotiq-3f-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; visual mesh filename=package://robotiq_3f_gripper_description/meshes/robotiq-3f-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
- link finger_2_link_0: geometry collision mesh filename=package://robotiq_3f_gripper_description/meshes/robotiq-3f-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; visual mesh filename=package://robotiq_3f_gripper_description/meshes/robotiq-3f-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
- link finger_2_link_1: geometry collision mesh filename=package://robotiq_3f_gripper_description/meshes/robotiq-3f-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; visual mesh filename=package://robotiq_3f_gripper_description/meshes/robotiq-3f-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
- link finger_2_link_2: geometry collision mesh filename=package://robotiq_3f_gripper_description/meshes/robotiq-3f-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; visual mesh filename=package://robotiq_3f_gripper_description/meshes/robotiq-3f-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
- link finger_2_link_3: geometry collision mesh filename=package://robotiq_3f_gripper_description/meshes/robotiq-3f-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; visual mesh filename=package://robotiq_3f_gripper_description/meshes/robotiq-3f-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
- link finger_middle_link_0: geometry collision mesh filename=package://robotiq_3f_gripper_description/meshes/robotiq-3f-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; visual mesh filename=package://robotiq_3f_gripper_description/meshes/robotiq-3f-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
- link finger_middle_link_1: geometry collision mesh filename=package://robotiq_3f_gripper_description/meshes/robotiq-3f-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; visual mesh filename=package://robotiq_3f_gripper_description/meshes/robotiq-3f-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
- link finger_middle_link_2: geometry collision mesh filename=package://robotiq_3f_gripper_description/meshes/robotiq-3f-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; visual mesh filename=package://robotiq_3f_gripper_description/meshes/robotiq-3f-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
- link finger_middle_link_3: geometry collision mesh filename=package://robotiq_3f_gripper_description/meshes/robotiq-3f-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; visual mesh filename=package://robotiq_3f_gripper_description/meshes/robotiq-3f-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
- link palm: geometry collision mesh filename=package://robotiq_3f_gripper_description/meshes/robotiq-3f-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; visual mesh filename=package://robotiq_3f_gripper_description/meshes/robotiq-3f-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

File: assets/end_effectors/robotiq_3f_gripper/robotiq_3f_gripper_description/urdf/robotiq-3f-gripper_articulated_macro.xacro (robot description, xacro)
@@ -15,5 +15,5 @@
 			<visual>
 				<geometry>
-                                        <mesh filename="package://robotiq_3f_gripper_visualization/meshes/robotiq-3f-gripper_articulated/visual/palm.dae" />
+                                        <mesh filename="package://robotiq_3f_gripper_description/meshes/robotiq-3f-gripper_articulated/visual/palm.dae" />
 				</geometry>
 				<material name="gray">
@@ -23,5 +23,5 @@
 			<collision>
 				<geometry>
-                                        <mesh filename="package://robotiq_3f_gripper_visualization/meshes/robotiq-3f-gripper_articulated/collision/palm.STL" />
+                                        <mesh filename="package://robotiq_3f_gripper_description/meshes/robotiq-3f-gripper_articulated/collision/palm.STL" />
 				</geometry>
 				<material name="yellow">

File: assets/end_effectors/robotiq_3f_gripper/robotiq_3f_gripper_description/urdf/robotiq-3f-gripper_finger_articulated_macro.xacro (robot description, xacro)
@@ -12,5 +12,5 @@
 				<origin xyz="0.020 0 0" rpy="0 0 0"/>
 				<geometry>
-                                        <mesh filename="package://robotiq_3f_gripper_visualization/meshes/robotiq-3f-gripper_articulated/visual/link_0.dae" />
+                                        <mesh filename="package://robotiq_3f_gripper_description/meshes/robotiq-3f-gripper_articulated/visual/link_0.dae" />
 				</geometry>
 				<material name="gray">
@@ -21,5 +21,5 @@
 				<origin xyz="0.020 0 0" rpy="0 0 0"/>
 				<geometry>
-                                        <mesh filename="package://robotiq_3f_gripper_visualization/meshes/robotiq-3f-gripper_articulated/collision/link_0.STL" />
+                                        <mesh filename="package://robotiq_3f_gripper_description/meshes/robotiq-3f-gripper_articulated/collision/link_0.STL" />
 				</geometry>
 				<material name="yellow">
@@ -37,5 +37,5 @@
 				<origin xyz="0.050 -.028 0" rpy="0 0 -0.52"/>
 				<geometry>
-                                        <mesh filename="package://robotiq_3f_gripper_visualization/meshes/robotiq-3f-gripper_articulated/visual/link_1.dae" />
+                                        <mesh filename="package://robotiq_3f_gripper_description/meshes/robotiq-3f-gripper_articulated/visual/link_1.dae" />
 				</geometry>
 				<material name="gray"/>
@@ -44,5 +44,5 @@
 				<origin xyz="0.050 -.028 0" rpy="0 0 -0.52"/>
 				<geometry>
-                                        <mesh filename="package://robotiq_3f_gripper_visualization/meshes/robotiq-3f-gripper_articulated/collision/link_1.STL" />
+                                        <mesh filename="package://robotiq_3f_gripper_description/meshes/robotiq-3f-gripper_articulated/collision/link_1.STL" />
 				</geometry>
 				<material name="yellow"/>
@@ -63,5 +63,5 @@
 				<origin xyz="0.039 0 0.0075" rpy="0 0 0"/>
 				<geometry>
-                                        <mesh filename="package://robotiq_3f_gripper_visualization/meshes/robotiq-3f-gripper_articulated/visual/link_2.dae" />
+                                        <mesh filename="package://robotiq_3f_gripper_description/meshes/robotiq-3f-gripper_articulated/visual/link_2.dae" />
 				</geometry>
 				<material name="gray"/>
@@ -70,5 +70,5 @@
 				<origin xyz="0.039 0 0.0075" rpy="0 0 0"/>
 				<geometry>
-                                        <mesh filename="package://robotiq_3f_gripper_visualization/meshes/robotiq-3f-gripper_articulated/collision/link_2.STL" />
+                                        <mesh filename="package://robotiq_3f_gripper_description/meshes/robotiq-3f-gripper_articulated/collision/link_2.STL" />
 				</geometry>
 				<material name="yellow"/>
@@ -84,5 +84,5 @@
 				<origin xyz="0 0 0" rpy="0 0 0.52"/>
 				<geometry>
-                                        <mesh filename="package://robotiq_3f_gripper_visualization/meshes/robotiq-3f-gripper_articulated/visual/link_3.dae" />
+                                        <mesh filename="package://robotiq_3f_gripper_description/meshes/robotiq-3f-gripper_articulated/visual/link_3.dae" />
 				</geometry>
 				<material name="gray"/>
@@ -91,5 +91,5 @@
 				<origin xyz="0 0 0" rpy="0 0 0.52"/>
 				<geometry>
-                                        <mesh filename="package://robotiq_3f_gripper_visualization/meshes/robotiq-3f-gripper_articulated/collision/link_3.STL" />
+                                        <mesh filename="package://robotiq_3f_gripper_description/meshes/robotiq-3f-gripper_articulated/collision/link_3.STL" />
 				</geometry>
 				<material name="yellow"/>

File: assets/end_effectors/robotiq_3f_gripper/robotiq_3f_gripper_description/urdf/robotiq-3f-gripper_mesh.urdf (robot description, URDF)
Before this commit: robot robotiq-3f-gripper_mesh, 4 links, 3 joints
Links:
- link finger_1: geometry collision mesh filename=package://robotiq_3f_gripper_description/meshes/robotiq-3f-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; visual mesh filename=package://robotiq_3f_gripper_description/meshes/robotiq-3f-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
- link finger_2: geometry collision mesh filename=package://robotiq_3f_gripper_description/meshes/robotiq-3f-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; visual mesh filename=package://robotiq_3f_gripper_description/meshes/robotiq-3f-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
- link finger_3: geometry collision mesh filename=package://robotiq_3f_gripper_description/meshes/robotiq-3f-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; visual mesh filename=package://robotiq_3f_gripper_description/meshes/robotiq-3f-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
- link palm: geometry collision mesh filename=package://robotiq_3f_gripper_description/meshes/robotiq-3f-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; visual mesh filename=package://robotiq_3f_gripper_description/meshes/robotiq-3f-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

File: assets/end_effectors/robotiq_3f_gripper/robotiq_3f_gripper_description/urdf/robotiq-3f-gripper_mesh_macro.xacro (robot description, xacro)
@@ -5,5 +5,5 @@
 			<visual>
 				<geometry>
-                                        <mesh filename="package://robotiq_3f_gripper_visualization/meshes/robotiq-3f-gripper/visual/GRIPPER_OPEN_PALM.stl" />
+                                        <mesh filename="package://robotiq_3f_gripper_description/meshes/robotiq-3f-gripper/visual/GRIPPER_OPEN_PALM.stl" />
 				</geometry>
 				<material name="green">
@@ -13,5 +13,5 @@
 			<collision>
 				<geometry>
-                                        <mesh filename="package://robotiq_3f_gripper_visualization/meshes/robotiq-3f-gripper/collision/GRIPPER_OPEN_PALM.stl" />
+                                        <mesh filename="package://robotiq_3f_gripper_description/meshes/robotiq-3f-gripper/collision/GRIPPER_OPEN_PALM.stl" />
 				</geometry>
 				<material name="yellow">
@@ -23,5 +23,5 @@
 			<visual>
 				<geometry>
-                                        <mesh filename="package://robotiq_3f_gripper_visualization/meshes/robotiq-3f-gripper/visual/GRIPPER_OPEN_FINGER_1.stl" />
+                                        <mesh filename="package://robotiq_3f_gripper_description/meshes/robotiq-3f-gripper/visual/GRIPPER_OPEN_FINGER_1.stl" />
 				</geometry>
 				<material name="green"/>
@@ -29,5 +29,5 @@
 			<collision>
 				<geometry>
-                                        <mesh filename="package://robotiq_3f_gripper_visualization/meshes/robotiq-3f-gripper/collision/GRIPPER_OPEN_FINGER_1.stl" />
+                                        <mesh filename="package://robotiq_3f_gripper_description/meshes/robotiq-3f-gripper/collision/GRIPPER_OPEN_FINGER_1.stl" />
 				</geometry>
 				<material name="yellow"/>
@@ -37,5 +37,5 @@
 			<visual>
 				<geometry>
-                                        <mesh filename="package://robotiq_3f_gripper_visualization/meshes/robotiq-3f-gripper/visual/GRIPPER_OPEN_FINGER_2.stl" />
+                                        <mesh filename="package://robotiq_3f_gripper_description/meshes/robotiq-3f-gripper/visual/GRIPPER_OPEN_FINGER_2.stl" />
 				</geometry>
 				<material name="green"/>
@@ -43,5 +43,5 @@
 			<collision>
 				<geometry>
-                                        <mesh filename="package://robotiq_3f_gripper_visualization/meshes/robotiq-3f-gripper/collision/GRIPPER_OPEN_FINGER_2.stl" />
+                                        <mesh filename="package://robotiq_3f_gripper_description/meshes/robotiq-3f-gripper/collision/GRIPPER_OPEN_FINGER_2.stl" />
 				</geometry>
 				<material name="yellow"/>
@@ -51,5 +51,5 @@
 			<visual>
 				<geometry>
-                                        <mesh filename="package://robotiq_3f_gripper_visualization/meshes/robotiq-3f-gripper/visual/GRIPPER_OPEN_FINGER_3.stl" />
+                                        <mesh filename="package://robotiq_3f_gripper_description/meshes/robotiq-3f-gripper/visual/GRIPPER_OPEN_FINGER_3.stl" />
 				</geometry>
 				<material name="green"/>
@@ -57,5 +57,5 @@
 			<collision>
 				<geometry>
-                                        <mesh filename="package://robotiq_3f_gripper_visualization/meshes/robotiq-3f-gripper/collision/GRIPPER_OPEN_FINGER_3.stl" />
+                                        <mesh filename="package://robotiq_3f_gripper_description/meshes/robotiq-3f-gripper/collision/GRIPPER_OPEN_FINGER_3.stl" />
 				</geometry>
 				<material name="yellow"/>

File: assets/end_effectors/robotiq_3f_gripper/robotiq_3f_gripper_description/urdf/robotiq_3f_hand_macro.urdf.xacro (robot description, xacro)
@@ -19,5 +19,5 @@
         <origin xyz="0 0 0" rpy="0 0 0"/>
         <geometry>
-          <mesh filename="package://robotiq_3f_gripper_visualization/meshes/robotiq-3f-gripper_articulated/visual/link_0.dae" />
+          <mesh filename="package://robotiq_3f_gripper_description/meshes/robotiq-3f-gripper_articulated/visual/link_0.dae" />
         </geometry>
         <material name="green">
@@ -28,5 +28,5 @@
         <origin rpy="0 0 0" xyz="0 0 0"/>
         <geometry>
-          <mesh filename="package://robotiq_3f_gripper_visualization/meshes/robotiq-3f-gripper_articulated/collision/link_0.STL" />
+          <mesh filename="package://robotiq_3f_gripper_description/meshes/robotiq-3f-gripper_articulated/collision/link_0.STL" />
         </geometry>
         <material name="yellow">
@@ -49,5 +49,5 @@
         <origin rpy="0 0 ${3.1416/2}" xyz="0 0.05717 0"/>
         <geometry>
-          <mesh filename="package://robotiq_3f_gripper_visualization/meshes/robotiq-3f-gripper_articulated/visual/link_1.dae" />
+          <mesh filename="package://robotiq_3f_gripper_description/meshes/robotiq-3f-gripper_articulated/visual/link_1.dae" />
         </geometry>
         <material name="green"/>
@@ -56,5 +56,5 @@
         <origin rpy="0 0 ${3.1416/2}" xyz="0 0.05717 0"/>
         <geometry>
-          <mesh filename="package://robotiq_3f_gripper_visualization/meshes/robotiq-3f-gripper_articulated/collision/link_1.STL"/>
+          <mesh filename="package://robotiq_3f_gripper_description/meshes/robotiq-3f-gripper_articulated/collision/link_1.STL"/>
         </geometry>
         <material name="yellow">
@@ -82,5 +82,5 @@
         <origin rpy="0 0 ${3.1416/2}" xyz="0 0.03810 0.0075"/>
         <geometry>
-          <mesh filename="package://robotiq_3f_gripper_visualization/meshes/robotiq-3f-gripper_articulated/visual/link_2.dae" />
+          <mesh filename="package://robotiq_3f_gripper_description/meshes/robotiq-3f-gripper_articulated/visual/link_2.dae" />
         </geometry>
         <material name="green"/>
@@ -89,5 +89,5 @@
         <origin rpy="0 0 ${3.1416/2}" xyz="0 0.03810 0.0075"/>
           <geometry>
-            <mesh filename="package://robotiq_3f_gripper_visualization/meshes/robotiq-3f-gripper_articulated/collision/link_2.STL"/>
+            <mesh filename="package://robotiq_3f_gripper_description/meshes/robotiq-3f-gripper_articulated/collision/link_2.STL"/>
           </geometry>
         <material name="yellow"/>
@@ -113,5 +113,5 @@
         <origin xyz="0 0 0" rpy="0 0 0"/>
         <geometry>
-          <mesh filename="package://robotiq_3f_gripper_visualization/meshes/robotiq-3f-gripper_articulated/visual/link_3.dae" />
+          <mesh filename="package://robotiq_3f_gripper_description/meshes/robotiq-3f-gripper_articulated/visual/link_3.dae" />
         </geometry>
         <material name="green"/>
@@ -120,5 +120,5 @@
         <origin xyz="0 0 0" rpy="0 0 0"/>
         <geometry>
-          <mesh filename="package://robotiq_3f_gripper_visualization/meshes/robotiq-3f-gripper_articulated/collision/link_3.STL"/>
+          <mesh filename="package://robotiq_3f_gripper_description/meshes/robotiq-3f-gripper_articulated/collision/link_3.STL"/>
         </geometry>
         <material name="yellow"/>
@@ -653,5 +653,5 @@
         <visual>
           <geometry>
-            <mesh filename="package://robotiq_3f_gripper_visualization/meshes/robotiq-3f-gripper_articulated/visual/palm.dae" />
+            <mesh filename="package://robotiq_3f_gripper_description/meshes/robotiq-3f-gripper_articulated/visual/palm.dae" />
           </geometry>
           <material name="green">
