Commit message: Align run_grasp_execution with arm-only UR5 scene config

File: scenes/ur5_3f_test/urdf/arm_hand.srdf.xacro (robot description, xacro)
@@ -2,25 +2,4 @@
 <robot xmlns:xacro="http://www.ros.org/wiki/xacro" name="ur5_3f_test">
   <xacro:include filename="$(find ur5_moveit_config)/config/ur5.srdf.xacro" />
-  <xacro:include filename="$(find robotiq_3f_moveit_config)/config/robotiq_3f_gripper.srdf.xacro"/>
   <xacro:ur5/>
-  <xacro:robotiq-3f-gripper_articulated/>
-  <disable_collisions link1="palm" link2="base_link" reason="Never" />
-  <disable_collisions link1="palm" link2="shoulder_link" reason="Never" />
-  <disable_collisions link1="palm" link2="upper_arm_link" reason="Never" />
-  <disable_collisions link1="palm" link2="forearm_link" reason="Never" />
-  <disable_collisions link1="palm" link2="wrist_1_link" reason="Never" />
-  <disable_collisions link1="palm" link2="wrist_2_link" reason="Never" />
-  <disable_collisions link1="palm" link2="wrist_3_link" reason="Never" />
-  <disable_collisions link1="palm" link2="tool0" reason="Never" />
-  <disable_collisions link1="palm" link2="base" reason="Never" />
-  <disable_collisions link1="palm" link2="tool0" reason="Never" />
-  <disable_collisions link1="finger_1_link_0" link2="wrist_3_link" reason="Never" />
-  <disable_collisions link1="finger_2_link_0" link2="wrist_3_link" reason="Never" />
-  <disable_collisions link1="finger_middle_link_0" link2="wrist_3_link" reason="Never" />
-  <disable_collisions link1="finger_1_link_0" link2="wrist_2_link" reason="Never" />
-  <disable_collisions link1="finger_2_link_0" link2="wrist_2_link" reason="Never" />
-  <disable_collisions link1="finger_middle_link_0" link2="wrist_2_link" reason="Never" />
-  <disable_collisions link1="finger_1_link_0" link2="tool0" reason="Never" />
-  <disable_collisions link1="finger_2_link_0" link2="tool0" reason="Never" />
-  <disable_collisions link1="finger_middle_link_0" link2="tool0" reason="Never" />
 </robot>

File: scenes/ur5_3f_test/urdf/scene.urdf.xacro (robot description, xacro)
@@ -19,12 +19,5 @@
   <origin xyz="0 0 0" rpy="0 0 0"/>
 </xacro:ur_robot>
- <!--xacro:include filename="$(find robotiq_85_description)/urdf/robotiq_85_gripper.urdf.xacro"/>
- <xacro:robotiq_85_gripper prefix="" parent="tool0">
-	<origin xyz="0 0 0" rpy="1.5707 -1.5707 0"/>
- </xacro:robotiq_85_gripper-->
- <xacro:include filename="$(find robotiq_3f_gripper_description)/urdf/robotiq-3f-gripper_articulated.urdf.xacro"/>
- <xacro:robotiq-3f-gripper_articulated prefix="" parent="tool0" >
-	<origin xyz="0 0 0.0" rpy="1.5707 0 0"/>
- </xacro:robotiq-3f-gripper_articulated>
+ <!-- Arm-only hardware variant: no physical gripper attached to tool0. -->
  <xacro:include filename="$(find workbench_description)/urdf/table.urdf.xacro"/>
  <xacro:table prefix="" parent="world">
