Commit message: Update UR5 xacro to ROS 2 driver macro

File: scenes/ur5_3f_test/urdf/scene.urdf.xacro (robot description, xacro)
@@ -2,6 +2,20 @@
 <robot xmlns:xacro="http://www.ros.org/wiki/xacro" name="ur5_3f_test">
  <link name="world"/>
- <xacro:include filename="$(find-pkg-share ur_description)/urdf/ur.urdf.xacro"/>
- <xacro:ur_robot prefix="" joint_limited="false" ur_type="ur5"/>
+ <xacro:include filename="$(find ur_description)/urdf/ur_macro.xacro"/>
+ <xacro:arg name="joint_limits_parameters_file" default="$(find ur_description)/config/ur5/joint_limits.yaml"/>
+ <xacro:arg name="kinematics_parameters_file" default="$(find ur_description)/config/ur5/default_kinematics.yaml"/>
+ <xacro:arg name="physical_parameters_file" default="$(find ur_description)/config/ur5/physical_parameters.yaml"/>
+ <xacro:arg name="visual_parameters_file" default="$(find ur_description)/config/ur5/visual_parameters.yaml"/>
+ <xacro:ur_robot
+   name="ur5"
+   tf_prefix=""
+   parent="world"
+   joint_limits_parameters_file="$(arg joint_limits_parameters_file)"
+   kinematics_parameters_file="$(arg kinematics_parameters_file)"
+   physical_parameters_file="$(arg physical_parameters_file)"
+   visual_parameters_file="$(arg visual_parameters_file)"
+   generate_ros2_control_tag="false">
+   <origin xyz="0 0 0" rpy="0 0 0" />
+ </xacro:ur_robot>
   <joint name="world_ur5" type="fixed">
 	<parent link="world" />

Commit message: Align ur5_3f_test tool contract

File: scenes/ur5_3f_test/urdf/scene.urdf.xacro (robot description, xacro)
@@ -19,5 +19,8 @@
   <origin xyz="0 0 0" rpy="0 0 0"/>
 </xacro:ur_robot>
- <!-- Arm-only hardware variant: no physical gripper attached to tool0. -->
+ <xacro:include filename="$(find robotiq_3f_gripper_description)/urdf/robotiq-3f-gripper_articulated.urdf.xacro"/>
+ <xacro:robotiq-3f-gripper_articulated prefix="" parent="tool0">
+	<origin xyz="0 0 0" rpy="0 0 0"/>
+ </xacro:robotiq-3f-gripper_articulated>
  <xacro:include filename="$(find workbench_description)/urdf/table.urdf.xacro"/>
  <xacro:table prefix="" parent="world">
@@ -31,7 +34,7 @@
  <link name="ee_palm" />
  <joint name="base_to_palm" type="fixed">
-    <parent link="tool0"/>
+    <parent link="palm"/>
     <child link="ee_palm"/>
-    <origin xyz="0 0 0.18" rpy="0 0 0"/>
+    <origin xyz="0 0 0.0875" rpy="0 0 0"/>
  </joint>
 </robot>
