Commit message: Fix ros2_control interfaces + add controllers yaml + update MoveIt octomap sensor params

File: assets/robots/universal_robot/ur5_moveit_config/config/ur5.ros2_control.xacro (robot description, xacro)
@@ -1,47 +1,84 @@
 <?xml version="1.0"?>
 <robot xmlns:xacro="http://www.ros.org/wiki/xacro">
-    <xacro:macro name="ur5_ros2_control" params="name initial_positions_file">
-        <xacro:property name="initial_positions" value="${xacro.load_yaml(initial_positions_file)['initial_positions']}"/>
-        <ros2_control name="${name}" type="system">
-            <hardware>
-                <plugin>fake_components/GenericSystem</plugin>
-            </hardware>
-            <joint name="shoulder_pan_joint">
-                <param name="initial_position">${initial_positions['shoulder_pan_joint']}</param>
-                <command_interface name="position" />
-                <state_interface name="position"/>
-                <state_interface name="velocity"/>
-            </joint>
-            <joint name="shoulder_lift_joint">
-                <param name="initial_position">${initial_positions['shoulder_lift_joint']}</param>
-                <command_interface name="position" />
-                <state_interface name="position"/>
-                <state_interface name="velocity"/>
-            </joint>
-            <joint name="elbow_joint">
-                <param name="initial_position">${initial_positions['elbow_joint']}</param>
-                <command_interface name="position" />
-                <state_interface name="position"/>
-                <state_interface name="velocity"/>
-            </joint>
-            <joint name="wrist_1_joint">
-                <param name="initial_position">${initial_positions['wrist_1_joint']}</param>
-                <command_interface name="position" />
-                <state_interface name="position"/>
-                <state_interface name="velocity"/>
-            </joint>
-            <joint name="wrist_2_joint">
-                <param name="initial_position">${initial_positions['wrist_2_joint']}</param>
-                <command_interface name="position" />
-                <state_interface name="position"/>
-                <state_interface name="velocity"/>
-            </joint>
-            <joint name="wrist_3_joint">
-                <param name="initial_position">${initial_positions['wrist_3_joint']}</param>
-                <command_interface name="position" />
-                <state_interface name="position"/>
-                <state_interface name="velocity"/>
-            </joint>
-        </ros2_control>
-    </xacro:macro>
+  <xacro:macro name="ur5_ros2_control" params="name initial_positions_file">
+    <xacro:property name="initial_positions"
+                    value="${xacro.load_yaml(initial_positions_file)['initial_positions']}"/>
+    <ros2_control name="${name}" type="system">
+      <hardware>
+        <plugin>fake_components/GenericSystem</plugin>
+      </hardware>
+      <!-- UR5 arm joints -->
+      <joint name="shoulder_pan_joint">
+        <param name="initial_position">${initial_positions['shoulder_pan_joint']}</param>
+        <command_interface name="position"/>
+        <state_interface name="position">
+          <param name="initial_value">${initial_positions['shoulder_pan_joint']}</param>
+        </state_interface>
+        <state_interface name="velocity">
+          <param name="initial_value">0.0</param>
+        </state_interface>
+      </joint>
+      <joint name="shoulder_lift_joint">
+        <param name="initial_position">${initial_positions['shoulder_lift_joint']}</param>
+        <command_interface name="position"/>
+        <state_interface name="position">
+          <param name="initial_value">${initial_positions['shoulder_lift_joint']}</param>
+        </state_interface>
+        <state_interface name="velocity">
+          <param name="initial_value">0.0</param>
+        </state_interface>
+      </joint>
+      <joint name="elbow_joint">
+        <param name="initial_position">${initial_positions['elbow_joint']}</param>
+        <command_interface name="position"/>
+        <state_interface name="position">
+          <param name="initial_value">${initial_positions['elbow_joint']}</param>
+        </state_interface>
+        <state_interface name="velocity">
+          <param name="initial_value">0.0</param>
+        </state_interface>
+      </joint>
+      <joint name="wrist_1_joint">
+        <param name="initial_position">${initial_positions['wrist_1_joint']}</param>
+        <command_interface name="position"/>
+        <state_interface name="position">
+          <param name="initial_value">${initial_positions['wrist_1_joint']}</param>
+        </state_interface>
+        <state_interface name="velocity">
+          <param name="initial_value">0.0</param>
+        </state_interface>
+      </joint>
+      <joint name="wrist_2_joint">
+        <param name="initial_position">${initial_positions['wrist_2_joint']}</param>
+        <command_interface name="position"/>
+        <state_interface name="position">
+          <param name="initial_value">${initial_positions['wrist_2_joint']}</param>
+        </state_interface>
+        <state_interface name="velocity">
+          <param name="initial_value">0.0</param>
+        </state_interface>
+      </joint>
+      <joint name="wrist_3_joint">
+        <param name="initial_position">${initial_positions['wrist_3_joint']}</param>
+        <command_interface name="position"/>
+        <state_interface name="position">
+          <param name="initial_value">${initial_positions['wrist_3_joint']}</param>
+        </state_interface>
+        <state_interface name="velocity">
+          <param name="initial_value">0.0</param>
+        </state_interface>
+      </joint>
+      <!-- Gripper (publish state so MoveIt stops complaining).
+           Use .get(..., 0.0) so you DON'T need to edit start_positions.yaml. -->
+      <joint name="gripper_finger1_joint">
+        <param name="initial_position">${initial_positions.get('gripper_finger1_joint', 0.0)}</param>
+        <state_interface name="position">
+          <param name="initial_value">${initial_positions.get('gripper_finger1_joint', 0.0)}</param>
+        </state_interface>
+        <state_interface name="velocity">
+          <param name="initial_value">0.0</param>
+        </state_interface>
+      </joint>
+    </ros2_control>
+  </xacro:macro>
 </robot>

Commit message: Add UR5 3F gripper ros2_control interfaces and joint-state validation

File: assets/robots/universal_robot/ur5_moveit_config/config/ur5.ros2_control.xacro (robot description, xacro)
@@ -43,4 +43,70 @@
                 <state_interface name="velocity"/>
             </joint>
+            <joint name="palm_finger_1_joint">
+                <param name="initial_position">0.0</param>
+                <command_interface name="position" />
+                <state_interface name="position"/>
+                <state_interface name="velocity"/>
+            </joint>
+            <joint name="finger_1_joint_1">
+                <param name="initial_position">0.0</param>
+                <command_interface name="position" />
+                <state_interface name="position"/>
+                <state_interface name="velocity"/>
+            </joint>
+            <joint name="finger_1_joint_2">
+                <param name="initial_position">0.0</param>
+                <command_interface name="position" />
+                <state_interface name="position"/>
+                <state_interface name="velocity"/>
+            </joint>
+            <joint name="finger_1_joint_3">
+                <param name="initial_position">0.0</param>
+                <command_interface name="position" />
+                <state_interface name="position"/>
+                <state_interface name="velocity"/>
+            </joint>
+            <joint name="palm_finger_2_joint">
+                <param name="initial_position">0.0</param>
+                <command_interface name="position" />
+                <state_interface name="position"/>
+                <state_interface name="velocity"/>
+            </joint>
+            <joint name="finger_2_joint_1">
+                <param name="initial_position">0.0</param>
+                <command_interface name="position" />
+                <state_interface name="position"/>
+                <state_interface name="velocity"/>
+            </joint>
+            <joint name="finger_2_joint_2">
+                <param name="initial_position">0.0</param>
+                <command_interface name="position" />
+                <state_interface name="position"/>
+                <state_interface name="velocity"/>
+            </joint>
+            <joint name="finger_2_joint_3">
+                <param name="initial_position">0.0</param>
+                <command_interface name="position" />
+                <state_interface name="position"/>
+                <state_interface name="velocity"/>
+            </joint>
+            <joint name="finger_middle_joint_1">
+                <param name="initial_position">0.0</param>
+                <command_interface name="position" />
+                <state_interface name="position"/>
+                <state_interface name="velocity"/>
+            </joint>
+            <joint name="finger_middle_joint_2">
+                <param name="initial_position">0.0</param>
+                <command_interface name="position" />
+                <state_interface name="position"/>
+                <state_interface name="velocity"/>
+            </joint>
+            <joint name="finger_middle_joint_3">
+                <param name="initial_position">0.0</param>
+                <command_interface name="position" />
+                <state_interface name="position"/>
+                <state_interface name="velocity"/>
+            </joint>
         </ros2_control>
     </xacro:macro>
