Commit message: Fix sorting scene realism and manifest frame consistency

File: scenes/ur5_2f_sorting_test/urdf/scene.urdf.xacro (robot description, xacro)
@@ -7,5 +7,5 @@
  <link name="world"/>
 <xacro:include filename="$(find ur_description)/urdf/ur_macro.xacro"/>
-<xacro:ur_robot
+ <xacro:ur_robot
   name="$(arg name)"
   tf_prefix="$(arg tf_prefix)"
@@ -17,5 +17,5 @@
   visual_parameters_file="$(find ur_description)/config/$(arg ur_type)/visual_parameters.yaml"
   use_fake_hardware="$(arg use_fake_hardware)">
-  <origin xyz="0 0 0" rpy="0 0 0"/>
+  <origin xyz="-0.55 0 0.76" rpy="0 0 0"/>
 </xacro:ur_robot>
  <xacro:include filename="$(find robotiq_85_description)/urdf/robotiq_85_gripper.urdf.xacro"/>
@@ -93,4 +93,20 @@
    <origin xyz="0.45 0.28 0.06" rpy="0 0 0"/>
  </joint>
+ <link name="reject_bin">
+   <visual>
+     <origin xyz="0 0 0" rpy="0 0 0"/>
+     <geometry><box size="0.22 0.18 0.12"/></geometry>
+     <material name="RejectBin"><color rgba="0.75 0.35 0.1 0.9"/></material>
+   </visual>
+   <collision>
+     <origin xyz="0 0 0" rpy="0 0 0"/>
+     <geometry><box size="0.22 0.18 0.12"/></geometry>
+   </collision>
+ </link>
+ <joint name="world_to_reject_bin" type="fixed">
+   <parent link="world"/>
+   <child link="reject_bin"/>
+   <origin xyz="0.20 0.36 0.06" rpy="0 0 0"/>
+ </joint>
  <link name="item_red">
    <visual><geometry><box size="0.04 0.04 0.08"/></geometry><material name="Red"><color rgba="0.9 0.1 0.1 1.0"/></material></visual>
@@ -100,5 +116,5 @@
    <parent link="world"/>
    <child link="item_red"/>
-   <origin xyz="0.30 -0.04 0.78" rpy="0 0 0"/>
+   <origin xyz="0.30 -0.04 0.80" rpy="0 0 0"/>
  </joint>
  <link name="item_blue">
@@ -109,5 +125,5 @@
    <parent link="world"/>
    <child link="item_blue"/>
-   <origin xyz="0.38 0.07 0.77" rpy="0 0 0"/>
+   <origin xyz="0.38 0.07 0.79" rpy="0 0 0"/>
  </joint>
  <link name="item_green">
@@ -118,5 +134,5 @@
    <parent link="world"/>
    <child link="item_green"/>
-   <origin xyz="0.34 0.12 0.765" rpy="0 0 0"/>
+   <origin xyz="0.34 0.12 0.775" rpy="0 0 0"/>
  </joint>
 </robot>

Commit message: Fix ur5 sorting scene physical layout realism

File: scenes/ur5_2f_sorting_test/urdf/scene.urdf.xacro (robot description, xacro)
@@ -6,4 +6,14 @@
  <xacro:arg name="use_fake_hardware" default="true"/>
  <link name="world"/>
+ <xacro:property name="table_top_z" value="0.76"/>
+ <xacro:property name="item_red_height" value="0.08"/>
+ <xacro:property name="item_blue_length" value="0.06"/>
+ <xacro:property name="item_green_radius" value="0.025"/>
+ <xacro:property name="tray_length" value="0.22"/>
+ <xacro:property name="tray_width" value="0.18"/>
+ <xacro:property name="tray_height" value="0.07"/>
+ <xacro:property name="pickup_area_x" value="0.30"/>
+ <xacro:property name="pickup_area_y" value="0.0"/>
+ <xacro:property name="destination_area_x" value="0.48"/>
 <xacro:include filename="$(find ur_description)/urdf/ur_macro.xacro"/>
  <xacro:ur_robot
@@ -17,5 +27,5 @@
   visual_parameters_file="$(find ur_description)/config/$(arg ur_type)/visual_parameters.yaml"
   use_fake_hardware="$(arg use_fake_hardware)">
-  <origin xyz="-0.55 0 0.76" rpy="0 0 0"/>
+  <origin xyz="-0.35 0.0 0.0" rpy="0 0 0"/>
 </xacro:ur_robot>
  <xacro:include filename="$(find robotiq_85_description)/urdf/robotiq_85_gripper.urdf.xacro"/>
@@ -63,11 +73,11 @@
  <link name="bin_a">
    <visual>
-     <origin xyz="0 0 0" rpy="0 0 0"/>
-     <geometry><box size="0.22 0.18 0.12"/></geometry>
+     <origin xyz="0 0 ${-tray_height / 2}" rpy="0 0 0"/>
+     <geometry><box size="${tray_length} ${tray_width} ${tray_height}"/></geometry>
      <material name="Blue"><color rgba="0.2 0.2 0.8 0.9"/></material>
    </visual>
    <collision>
-     <origin xyz="0 0 0" rpy="0 0 0"/>
-     <geometry><box size="0.22 0.18 0.12"/></geometry>
+     <origin xyz="0 0 ${-tray_height / 2}" rpy="0 0 0"/>
+     <geometry><box size="${tray_length} ${tray_width} ${tray_height}"/></geometry>
    </collision>
  </link>
@@ -75,15 +85,15 @@
    <parent link="world"/>
    <child link="bin_a"/>
-   <origin xyz="0.45 -0.28 0.06" rpy="0 0 0"/>
+   <origin xyz="${destination_area_x} -0.25 ${table_top_z + tray_height}" rpy="0 0 0"/>
  </joint>
  <link name="bin_b">
    <visual>
-     <origin xyz="0 0 0" rpy="0 0 0"/>
-     <geometry><box size="0.22 0.18 0.12"/></geometry>
+     <origin xyz="0 0 ${-tray_height / 2}" rpy="0 0 0"/>
+     <geometry><box size="${tray_length} ${tray_width} ${tray_height}"/></geometry>
      <material name="Green"><color rgba="0.2 0.8 0.2 0.9"/></material>
    </visual>
    <collision>
-     <origin xyz="0 0 0" rpy="0 0 0"/>
-     <geometry><box size="0.22 0.18 0.12"/></geometry>
+     <origin xyz="0 0 ${-tray_height / 2}" rpy="0 0 0"/>
+     <geometry><box size="${tray_length} ${tray_width} ${tray_height}"/></geometry>
    </collision>
  </link>
@@ -91,15 +101,15 @@
    <parent link="world"/>
    <child link="bin_b"/>
-   <origin xyz="0.45 0.28 0.06" rpy="0 0 0"/>
+   <origin xyz="${destination_area_x} 0.0 ${table_top_z + tray_height}" rpy="0 0 0"/>
  </joint>
  <link name="reject_bin">
    <visual>
-     <origin xyz="0 0 0" rpy="0 0 0"/>
-     <geometry><box size="0.22 0.18 0.12"/></geometry>
+     <origin xyz="0 0 ${-tray_height / 2}" rpy="0 0 0"/>
+     <geometry><box size="${tray_length} ${tray_width} ${tray_height}"/></geometry>
      <material name="RejectBin"><color rgba="0.75 0.35 0.1 0.9"/></material>
    </visual>
    <collision>
-     <origin xyz="0 0 0" rpy="0 0 0"/>
-     <geometry><box size="0.22 0.18 0.12"/></geometry>
+     <origin xyz="0 0 ${-tray_height / 2}" rpy="0 0 0"/>
+     <geometry><box size="${tray_length} ${tray_width} ${tray_height}"/></geometry>
    </collision>
  </link>
@@ -107,5 +117,5 @@
    <parent link="world"/>
    <child link="reject_bin"/>
-   <origin xyz="0.20 0.36 0.06" rpy="0 0 0"/>
+   <origin xyz="${destination_area_x} 0.25 ${table_top_z + tray_height}" rpy="0 0 0"/>
  </joint>
  <link name="item_red">
@@ -116,5 +126,5 @@
    <parent link="world"/>
    <child link="item_red"/>
-   <origin xyz="0.30 -0.04 0.80" rpy="0 0 0"/>
+   <origin xyz="${pickup_area_x} ${pickup_area_y - 0.10} ${table_top_z + item_red_height / 2}" rpy="0 0 0"/>
  </joint>
  <link name="item_blue">
@@ -125,5 +135,5 @@
    <parent link="world"/>
    <child link="item_blue"/>
-   <origin xyz="0.38 0.07 0.79" rpy="0 0 0"/>
+   <origin xyz="${pickup_area_x + 0.08} ${pickup_area_y} ${table_top_z + item_blue_length / 2}" rpy="0 0 0"/>
  </joint>
  <link name="item_green">
@@ -134,5 +144,5 @@
    <parent link="world"/>
    <child link="item_green"/>
-   <origin xyz="0.34 0.12 0.775" rpy="0 0 0"/>
+   <origin xyz="${pickup_area_x + 0.04} ${pickup_area_y + 0.10} ${table_top_z + item_green_radius}" rpy="0 0 0"/>
  </joint>
 </robot>

Commit message: Fix sorting scene with deterministic local table layout

File: scenes/ur5_2f_sorting_test/urdf/scene.urdf.xacro (robot description, xacro)
@@ -6,15 +6,63 @@
  <xacro:arg name="use_fake_hardware" default="true"/>
  <link name="world"/>
- <xacro:property name="table_top_z" value="0.76"/>
+ <xacro:property name="floor_z" value="0.0"/>
+ <xacro:property name="table_length" value="1.20"/>
+ <xacro:property name="table_width" value="0.70"/>
+ <xacro:property name="table_height" value="0.74"/>
+ <xacro:property name="table_top_thickness" value="0.04"/>
+ <xacro:property name="table_top_z" value="${floor_z + table_height}"/>
+ <xacro:property name="tray_length" value="0.22"/>
+ <xacro:property name="tray_width" value="0.18"/>
+ <xacro:property name="tray_height" value="0.07"/>
  <xacro:property name="item_red_height" value="0.08"/>
  <xacro:property name="item_blue_length" value="0.06"/>
  <xacro:property name="item_green_radius" value="0.025"/>
- <xacro:property name="tray_length" value="0.22"/>
- <xacro:property name="tray_width" value="0.18"/>
- <xacro:property name="tray_height" value="0.07"/>
- <xacro:property name="pickup_area_x" value="0.30"/>
+ <xacro:property name="pickup_area_x" value="0.32"/>
  <xacro:property name="pickup_area_y" value="0.0"/>
- <xacro:property name="destination_area_x" value="0.48"/>
-<xacro:include filename="$(find ur_description)/urdf/ur_macro.xacro"/>
+ <xacro:property name="destination_area_x" value="0.50"/>
+ <xacro:property name="table_leg_size" value="0.07"/>
+ <xacro:property name="robot_plate_length" value="0.28"/>
+ <xacro:property name="robot_plate_width" value="0.28"/>
+ <xacro:property name="robot_plate_thickness" value="0.03"/>
+ <xacro:include filename="$(find ur_description)/urdf/ur_macro.xacro"/>
+ <link name="table_">
+   <visual>
+     <origin xyz="0 0 ${-(table_height - table_top_thickness) / 2}" rpy="0 0 0"/>
+     <geometry><box size="${table_length} ${table_width} ${table_height - table_top_thickness}"/></geometry>
+     <material name="TableCabinet"><color rgba="0.46 0.33 0.24 1.0"/></material>
+   </visual>
+   <collision>
+     <origin xyz="0 0 ${-(table_height - table_top_thickness) / 2}" rpy="0 0 0"/>
+     <geometry><box size="${table_length} ${table_width} ${table_height - table_top_thickness}"/></geometry>
+   </collision>
+   <visual>
+     <origin xyz="0 0 ${table_top_thickness / 2}" rpy="0 0 0"/>
+     <geometry><box size="${table_length} ${table_width} ${table_top_thickness}"/></geometry>
+     <material name="TableTop"><color rgba="0.55 0.40 0.28 1.0"/></material>
+   </visual>
+   <collision>
+     <origin xyz="0 0 ${table_top_thickness / 2}" rpy="0 0 0"/>
+     <geometry><box size="${table_length} ${table_width} ${table_top_thickness}"/></geometry>
+   </collision>
+ </link>
+ <joint name="world_to_table" type="fixed">
+   <parent link="world"/>
+   <child link="table_"/>
+   <origin xyz="0.15 0 ${table_top_z}" rpy="0 0 0"/>
+ </joint>
+ <link name="robot_mount_plate">
+   <visual>
+     <geometry><box size="${robot_plate_length} ${robot_plate_width} ${robot_plate_thickness}"/></geometry>
+     <material name="RobotPlate"><color rgba="0.25 0.25 0.25 1.0"/></material>
+   </visual>
+   <collision>
+     <geometry><box size="${robot_plate_length} ${robot_plate_width} ${robot_plate_thickness}"/></geometry>
+   </collision>
+ </link>
+ <joint name="table_to_robot_mount_plate" type="fixed">
+   <parent link="table_"/>
+   <child link="robot_mount_plate"/>
+   <origin xyz="-0.44 0.0 ${robot_plate_thickness / 2}" rpy="0 0 0"/>
+ </joint>
  <xacro:ur_robot
   name="$(arg name)"
@@ -27,9 +75,9 @@
   visual_parameters_file="$(find ur_description)/config/$(arg ur_type)/visual_parameters.yaml"
   use_fake_hardware="$(arg use_fake_hardware)">
-  <origin xyz="-0.35 0.0 0.0" rpy="0 0 0"/>
-</xacro:ur_robot>
+  <origin xyz="-0.29 0.0 ${table_top_z + robot_plate_thickness}" rpy="0 0 0"/>
+ </xacro:ur_robot>
  <xacro:include filename="$(find robotiq_85_description)/urdf/robotiq_85_gripper.urdf.xacro"/>
  <xacro:robotiq_85_gripper prefix="" parent="tool0">
-	<origin xyz="0 0 0" rpy="1.5707 -1.5707 0"/>
+ 	<origin xyz="0 0 0" rpy="1.5707 -1.5707 0"/>
  </xacro:robotiq_85_gripper>
  <xacro:if value="$(arg use_fake_hardware)">
@@ -49,12 +97,8 @@
    </ros2_control>
  </xacro:if>
- <xacro:include filename="$(find workbench_description)/urdf/table.urdf.xacro"/>
- <xacro:table prefix="" parent="world">
-	<origin xyz="0 0 0" rpy="0 0 0"/>
- </xacro:table>
  <xacro:include filename="$(find realsense2_description)/urdf/_d435i.urdf.xacro"/>
  <xacro:arg name="use_nominal_extrinsics" default="true" />
  <xacro:sensor_d435i parent="table_" use_nominal_extrinsics="$(arg use_nominal_extrinsics)">
-    <origin xyz="-0.58 0.12 0.655" rpy="0 1.57079506 0"/>
+    <origin xyz="-0.58 0.12 0.62" rpy="0 1.57079506 0"/>
  </xacro:sensor_d435i>
  <link name="camera_frame" />
@@ -62,5 +106,4 @@
     <parent link="camera_link"/>
     <child link="camera_frame"/>
-    <!--origin xyz="0 0 0" rpy="0 0 3.14159"/-->
     <origin xyz="0 0 0" rpy="1.57079506 0 1.57079506"/>
  </joint>

Commit message: Polish ur5 sorting scene visuals and layout validation

File: scenes/ur5_2f_sorting_test/urdf/scene.urdf.xacro (robot description, xacro)
@@ -15,10 +15,11 @@
  <xacro:property name="tray_width" value="0.18"/>
  <xacro:property name="tray_height" value="0.07"/>
+ <xacro:property name="tray_wall_thickness" value="0.01"/>
  <xacro:property name="item_red_height" value="0.08"/>
  <xacro:property name="item_blue_length" value="0.06"/>
  <xacro:property name="item_green_radius" value="0.025"/>
- <xacro:property name="pickup_area_x" value="0.32"/>
- <xacro:property name="pickup_area_y" value="0.0"/>
- <xacro:property name="destination_area_x" value="0.50"/>
+ <xacro:property name="pickup_area_x" value="0.28"/>
+ <xacro:property name="pickup_area_y" value="-0.12"/>
+ <xacro:property name="destination_area_x" value="0.44"/>
  <xacro:property name="table_leg_size" value="0.07"/>
  <xacro:property name="robot_plate_length" value="0.28"/>
@@ -26,4 +27,5 @@
  <xacro:property name="robot_plate_thickness" value="0.03"/>
  <xacro:include filename="$(find ur_description)/urdf/ur_macro.xacro"/>
+ <!-- Workbench frame: table_ is the main contact link; top surface z is table_top_z. -->
  <link name="table_">
    <visual>
@@ -114,13 +116,46 @@
     <origin xyz="0 0 0.14" rpy="0 0 0"/>
  </joint>
+ <!-- Sorting destination row: tray frames are at opening/top-center; geometry extends downward onto tabletop. -->
  <link name="bin_a">
    <visual>
-     <origin xyz="0 0 ${-tray_height / 2}" rpy="0 0 0"/>
-     <geometry><box size="${tray_length} ${tray_width} ${tray_height}"/></geometry>
-     <material name="Blue"><color rgba="0.2 0.2 0.8 0.9"/></material>
-   </visual>
-   <collision>
-     <origin xyz="0 0 ${-tray_height / 2}" rpy="0 0 0"/>
-     <geometry><box size="${tray_length} ${tray_width} ${tray_height}"/></geometry>
+     <origin xyz="0 0 ${-tray_wall_thickness / 2}" rpy="0 0 0"/>
+     <geometry><box size="${tray_length} ${tray_width} ${tray_wall_thickness}"/></geometry>
+     <material name="Blue"><color rgba="0.2 0.2 0.8 1.0"/></material>
+   </visual>
+   <collision>
+     <origin xyz="0 0 ${-tray_wall_thickness / 2}" rpy="0 0 0"/>
+     <geometry><box size="${tray_length} ${tray_width} ${tray_wall_thickness}"/></geometry>
+   </collision>
+   <visual>
+     <origin xyz="0 ${tray_width / 2 - tray_wall_thickness / 2} ${-tray_height / 2}" rpy="0 0 0"/>
+     <geometry><box size="${tray_length} ${tray_wall_thickness} ${tray_height}"/></geometry>
+   </visual>
+   <collision>
+     <origin xyz="0 ${tray_width / 2 - tray_wall_thickness / 2} ${-tray_height / 2}" rpy="0 0 0"/>
+     <geometry><box size="${tray_length} ${tray_wall_thickness} ${tray_height}"/></geometry>
+   </collision>
+   <visual>
+     <origin xyz="0 ${-tray_width / 2 + tray_wall_thickness / 2} ${-tray_height / 2}" rpy="0 0 0"/>
+     <geometry><box size="${tray_length} ${tray_wall_thickness} ${tray_height}"/></geometry>
+   </visual>
+   <collision>
+     <origin xyz="0 ${-tray_width / 2 + tray_wall_thickness / 2} ${-tray_height / 2}" rpy="0 0 0"/>
+     <geometry><box size="${tray_length} ${tray_wall_thickness} ${tray_height}"/></geometry>
+   </collision>
+   <visual>
+     <origin xyz="${tray_length / 2 - tray_wall_thickness / 2} 0 ${-tray_height / 2}" rpy="0 0 0"/>
+     <geometry><box size="${tray_wall_thickness} ${tray_width} ${tray_height}"/></geometry>
+   </visual>
+   <collision>
+     <origin xyz="${tray_length / 2 - tray_wall_thickness / 2} 0 ${-tray_height / 2}" rpy="0 0 0"/>
+     <geometry><box size="${tray_wall_thickness} ${tray_width} ${tray_height}"/></geometry>
+   </collision>
+   <visual>
+     <origin xyz="${-tray_length / 2 + tray_wall_thickness / 2} 0 ${-tray_height / 2}" rpy="0 0 0"/>
+     <geometry><box size="${tray_wall_thickness} ${tray_width} ${tray_height}"/></geometry>
+   </visual>
+   <collision>
+     <origin xyz="${-tray_length / 2 + tray_wall_thickness / 2} 0 ${-tray_height / 2}" rpy="0 0 0"/>
+     <geometry><box size="${tray_wall_thickness} ${tray_width} ${tray_height}"/></geometry>
    </collision>
  </link>
@@ -128,38 +163,45 @@
    <parent link="world"/>
    <child link="bin_a"/>
-   <origin xyz="${destination_area_x} -0.25 ${table_top_z + tray_height}" rpy="0 0 0"/>
+   <origin xyz="${destination_area_x} -0.24 ${table_top_z + tray_wall_thickness}" rpy="0 0 0"/>
  </joint>
  <link name="bin_b">
    <visual>
-     <origin xyz="0 0 ${-tray_height / 2}" rpy="0 0 0"/>
-     <geometry><box size="${tray_length} ${tray_width} ${tray_height}"/></geometry>
-     <material name="Green"><color rgba="0.2 0.8 0.2 0.9"/></material>
-   </visual>
-   <collision>
-     <origin xyz="0 0 ${-tray_height / 2}" rpy="0 0 0"/>
-     <geometry><box size="${tray_length} ${tray_width} ${tray_height}"/></geometry>
-   </collision>
+     <origin xyz="0 0 ${-tray_wall_thickness / 2}" rpy="0 0 0"/>
+     <geometry><box size="${tray_length} ${tray_width} ${tray_wall_thickness}"/></geometry>
+     <material name="Green"><color rgba="0.2 0.8 0.2 1.0"/></material>
+   </visual>
+   <collision><origin xyz="0 0 ${-tray_wall_thickness / 2}" rpy="0 0 0"/><geometry><box size="${tray_length} ${tray_width} ${tray_wall_thickness}"/></geometry></collision>
+   <visual><origin xyz="0 ${tray_width / 2 - tray_wall_thickness / 2} ${-tray_height / 2}" rpy="0 0 0"/><geometry><box size="${tray_length} ${tray_wall_thickness} ${tray_height}"/></geometry></visual>
+   <collision><origin xyz="0 ${tray_width / 2 - tray_wall_thickness / 2} ${-tray_height / 2}" rpy="0 0 0"/><geometry><box size="${tray_length} ${tray_wall_thickness} ${tray_height}"/></geometry></collision>
+   <visual><origin xyz="0 ${-tray_width / 2 + tray_wall_thickness / 2} ${-tray_height / 2}" rpy="0 0 0"/><geometry><box size="${tray_length} ${tray_wall_thickness} ${tray_height}"/></geometry></visual>
+   <collision><origin xyz="0 ${-tray_width / 2 + tray_wall_thickness / 2} ${-tray_height / 2}" rpy="0 0 0"/><geometry><box size="${tray_length} ${tray_wall_thickness} ${tray_height}"/></geometry></collision>
+   <visual><origin xyz="${tray_length / 2 - tray_wall_thickness / 2} 0 ${-tray_height / 2}" rpy="0 0 0"/><geometry><box size="${tray_wall_thickness} ${tray_width} ${tray_height}"/></geometry></visual>
+   <collision><origin xyz="${tray_length / 2 - tray_wall_thickness / 2} 0 ${-tray_height / 2}" rpy="0 0 0"/><geometry><box size="${tray_wall_thickness} ${tray_width} ${tray_height}"/></geometry></collision>
+   <visual><origin xyz="${-tray_length / 2 + tray_wall_thickness / 2} 0 ${-tray_height / 2}" rpy="0 0 0"/><geometry><box size="${tray_wall_thickness} ${tray_width} ${tray_height}"/></geometry></visual>
+   <collision><origin xyz="${-tray_length / 2 + tray_wall_thickness / 2} 0 ${-tray_height / 2}" rpy="0 0 0"/><geometry><box size="${tray_wall_thickness} ${tray_width} ${tray_height}"/></geometry></collision>
  </link>
  <joint name="world_to_bin_b" type="fixed">
    <parent link="world"/>
    <child link="bin_b"/>
-   <origin xyz="${destination_area_x} 0.0 ${table_top_z + tray_height}" rpy="0 0 0"/>
+   <origin xyz="${destination_area_x} 0.0 ${table_top_z + tray_wall_thickness}" rpy="0 0 0"/>
  </joint>
  <link name="reject_bin">
-   <visual>
-     <origin xyz="0 0 ${-tray_height / 2}" rpy="0 0 0"/>
-     <geometry><box size="${tray_length} ${tray_width} ${tray_height}"/></geometry>
-     <material name="RejectBin"><color rgba="0.75 0.35 0.1 0.9"/></material>
-   </visual>
-   <collision>
-     <origin xyz="0 0 ${-tray_height / 2}" rpy="0 0 0"/>
-     <geometry><box size="${tray_length} ${tray_width} ${tray_height}"/></geometry>
-   </collision>
+   <visual><origin xyz="0 0 ${-tray_wall_thickness / 2}" rpy="0 0 0"/><geometry><box size="${tray_length} ${tray_width} ${tray_wall_thickness}"/></geometry><material name="RejectBin"><color rgba="0.75 0.35 0.1 1.0"/></material></visual>
+   <collision><origin xyz="0 0 ${-tray_wall_thickness / 2}" rpy="0 0 0"/><geometry><box size="${tray_length} ${tray_width} ${tray_wall_thickness}"/></geometry></collision>
+   <visual><origin xyz="0 ${tray_width / 2 - tray_wall_thickness / 2} ${-tray_height / 2}" rpy="0 0 0"/><geometry><box size="${tray_length} ${tray_wall_thickness} ${tray_height}"/></geometry></visual>
+   <collision><origin xyz="0 ${tray_width / 2 - tray_wall_thickness / 2} ${-tray_height / 2}" rpy="0 0 0"/><geometry><box size="${tray_length} ${tray_wall_thickness} ${tray_height}"/></geometry></collision>
+   <visual><origin xyz="0 ${-tray_width / 2 + tray_wall_thickness / 2} ${-tray_height / 2}" rpy="0 0 0"/><geometry><box size="${tray_length} ${tray_wall_thickness} ${tray_height}"/></geometry></visual>
+   <collision><origin xyz="0 ${-tray_width / 2 + tray_wall_thickness / 2} ${-tray_height / 2}" rpy="0 0 0"/><geometry><box size="${tray_length} ${tray_wall_thickness} ${tray_height}"/></geometry></collision>
+   <visual><origin xyz="${tray_length / 2 - tray_wall_thickness / 2} 0 ${-tray_height / 2}" rpy="0 0 0"/><geometry><box size="${tray_wall_thickness} ${tray_width} ${tray_height}"/></geometry></visual>
+   <collision><origin xyz="${tray_length / 2 - tray_wall_thickness / 2} 0 ${-tray_height / 2}" rpy="0 0 0"/><geometry><box size="${tray_wall_thickness} ${tray_width} ${tray_height}"/></geometry></collision>
+   <visual><origin xyz="${-tray_length / 2 + tray_wall_thickness / 2} 0 ${-tray_height / 2}" rpy="0 0 0"/><geometry><box size="${tray_wall_thickness} ${tray_width} ${tray_height}"/></geometry></visual>
+   <collision><origin xyz="${-tray_length / 2 + tray_wall_thickness / 2} 0 ${-tray_height / 2}" rpy="0 0 0"/><geometry><box size="${tray_wall_thickness} ${tray_width} ${tray_height}"/></geometry></collision>
  </link>
  <joint name="world_to_reject_bin" type="fixed">
    <parent link="world"/>
    <child link="reject_bin"/>
-   <origin xyz="${destination_area_x} 0.25 ${table_top_z + tray_height}" rpy="0 0 0"/>
- </joint>
+   <origin xyz="${destination_area_x} 0.24 ${table_top_z + tray_wall_thickness}" rpy="0 0 0"/>
+ </joint>
+ <!-- Pickup area: three items arranged in a reachable row on the tabletop (bottoms at table_top_z). -->
  <link name="item_red">
    <visual><geometry><box size="0.04 0.04 0.08"/></geometry><material name="Red"><color rgba="0.9 0.1 0.1 1.0"/></material></visual>
@@ -169,5 +211,5 @@
    <parent link="world"/>
    <child link="item_red"/>
-   <origin xyz="${pickup_area_x} ${pickup_area_y - 0.10} ${table_top_z + item_red_height / 2}" rpy="0 0 0"/>
+   <origin xyz="${pickup_area_x} ${pickup_area_y} ${table_top_z + item_red_height / 2}" rpy="0 0 0"/>
  </joint>
  <link name="item_blue">
@@ -187,5 +229,5 @@
    <parent link="world"/>
    <child link="item_green"/>
-   <origin xyz="${pickup_area_x + 0.04} ${pickup_area_y + 0.10} ${table_top_z + item_green_radius}" rpy="0 0 0"/>
+   <origin xyz="${pickup_area_x + 0.16} ${pickup_area_y} ${table_top_z + item_green_radius}" rpy="0 0 0"/>
  </joint>
 </robot>
