Commit message: Fix sorting scene tabletop/tray frames and validator parsing

File: scenes/ur5_2f_sorting_test/urdf/scene.urdf.xacro (robot description, xacro)
@@ -27,5 +27,5 @@
  <xacro:property name="robot_plate_thickness" value="0.03"/>
  <xacro:include filename="$(find ur_description)/urdf/ur_macro.xacro"/>
- <!-- Workbench frame: table_ is the main contact link; top surface z is table_top_z. -->
+ <!-- Workbench frame semantics: table_ frame is tabletop top-surface center (z=0 at top). -->
  <link name="table_">
    <visual>
@@ -39,10 +39,10 @@
    </collision>
    <visual>
-     <origin xyz="0 0 ${table_top_thickness / 2}" rpy="0 0 0"/>
+     <origin xyz="0 0 ${-table_top_thickness / 2}" rpy="0 0 0"/>
      <geometry><box size="${table_length} ${table_width} ${table_top_thickness}"/></geometry>
      <material name="TableTop"><color rgba="0.55 0.40 0.28 1.0"/></material>
    </visual>
    <collision>
-     <origin xyz="0 0 ${table_top_thickness / 2}" rpy="0 0 0"/>
+     <origin xyz="0 0 ${-table_top_thickness / 2}" rpy="0 0 0"/>
      <geometry><box size="${table_length} ${table_width} ${table_top_thickness}"/></geometry>
    </collision>
@@ -101,6 +101,22 @@
  <xacro:include filename="$(find realsense2_description)/urdf/_d435i.urdf.xacro"/>
  <xacro:arg name="use_nominal_extrinsics" default="true" />
+ <link name="camera_mast">
+   <visual>
+     <origin xyz="0 0 0.32" rpy="0 0 0"/>
+     <geometry><cylinder radius="0.01" length="0.64"/></geometry>
+     <material name="CameraMast"><color rgba="0.2 0.2 0.2 1.0"/></material>
+   </visual>
+   <collision>
+     <origin xyz="0 0 0.32" rpy="0 0 0"/>
+     <geometry><cylinder radius="0.01" length="0.64"/></geometry>
+   </collision>
+ </link>
+ <joint name="table_to_camera_mast" type="fixed">
+   <parent link="table_"/>
+   <child link="camera_mast"/>
+   <origin xyz="-0.18 0.28 0.0" rpy="0 0 0"/>
+ </joint>
  <xacro:sensor_d435i parent="table_" use_nominal_extrinsics="$(arg use_nominal_extrinsics)">
-    <origin xyz="-0.58 0.12 0.62" rpy="0 1.57079506 0"/>
+    <origin xyz="-0.18 0.10 0.62" rpy="0 1.57079506 0"/>
  </xacro:sensor_d435i>
  <link name="camera_frame" />
@@ -119,10 +135,10 @@
  <link name="bin_a">
    <visual>
-     <origin xyz="0 0 ${-tray_wall_thickness / 2}" rpy="0 0 0"/>
+     <origin xyz="0 0 ${-tray_height + tray_wall_thickness / 2}" rpy="0 0 0"/>
      <geometry><box size="${tray_length} ${tray_width} ${tray_wall_thickness}"/></geometry>
      <material name="Blue"><color rgba="0.2 0.2 0.8 1.0"/></material>
    </visual>
    <collision>
-     <origin xyz="0 0 ${-tray_wall_thickness / 2}" rpy="0 0 0"/>
+     <origin xyz="0 0 ${-tray_height + tray_wall_thickness / 2}" rpy="0 0 0"/>
      <geometry><box size="${tray_length} ${tray_width} ${tray_wall_thickness}"/></geometry>
    </collision>
@@ -160,16 +176,16 @@
    </collision>
  </link>
- <joint name="world_to_bin_a" type="fixed">
-   <parent link="world"/>
+ <joint name="table_to_bin_a" type="fixed">
+   <parent link="table_"/>
    <child link="bin_a"/>
-   <origin xyz="${destination_area_x} -0.24 ${table_top_z + tray_wall_thickness}" rpy="0 0 0"/>
+   <origin xyz="${destination_area_x} -0.24 ${tray_height}" rpy="0 0 0"/>
  </joint>
  <link name="bin_b">
    <visual>
-     <origin xyz="0 0 ${-tray_wall_thickness / 2}" rpy="0 0 0"/>
+     <origin xyz="0 0 ${-tray_height + tray_wall_thickness / 2}" rpy="0 0 0"/>
      <geometry><box size="${tray_length} ${tray_width} ${tray_wall_thickness}"/></geometry>
      <material name="Green"><color rgba="0.2 0.8 0.2 1.0"/></material>
    </visual>
-   <collision><origin xyz="0 0 ${-tray_wall_thickness / 2}" rpy="0 0 0"/><geometry><box size="${tray_length} ${tray_width} ${tray_wall_thickness}"/></geometry></collision>
+   <collision><origin xyz="0 0 ${-tray_height + tray_wall_thickness / 2}" rpy="0 0 0"/><geometry><box size="${tray_length} ${tray_width} ${tray_wall_thickness}"/></geometry></collision>
    <visual><origin xyz="0 ${tray_width / 2 - tray_wall_thickness / 2} ${-tray_height / 2}" rpy="0 0 0"/><geometry><box size="${tray_length} ${tray_wall_thickness} ${tray_height}"/></geometry></visual>
    <collision><origin xyz="0 ${tray_width / 2 - tray_wall_thickness / 2} ${-tray_height / 2}" rpy="0 0 0"/><geometry><box size="${tray_length} ${tray_wall_thickness} ${tray_height}"/></geometry></collision>
@@ -181,12 +197,12 @@
    <collision><origin xyz="${-tray_length / 2 + tray_wall_thickness / 2} 0 ${-tray_height / 2}" rpy="0 0 0"/><geometry><box size="${tray_wall_thickness} ${tray_width} ${tray_height}"/></geometry></collision>
  </link>
- <joint name="world_to_bin_b" type="fixed">
-   <parent link="world"/>
+ <joint name="table_to_bin_b" type="fixed">
+   <parent link="table_"/>
    <child link="bin_b"/>
-   <origin xyz="${destination_area_x} 0.0 ${table_top_z + tray_wall_thickness}" rpy="0 0 0"/>
+   <origin xyz="${destination_area_x} 0.0 ${tray_height}" rpy="0 0 0"/>
  </joint>
  <link name="reject_bin">
-   <visual><origin xyz="0 0 ${-tray_wall_thickness / 2}" rpy="0 0 0"/><geometry><box size="${tray_length} ${tray_width} ${tray_wall_thickness}"/></geometry><material name="RejectBin"><color rgba="0.75 0.35 0.1 1.0"/></material></visual>
-   <collision><origin xyz="0 0 ${-tray_wall_thickness / 2}" rpy="0 0 0"/><geometry><box size="${tray_length} ${tray_width} ${tray_wall_thickness}"/></geometry></collision>
+   <visual><origin xyz="0 0 ${-tray_height + tray_wall_thickness / 2}" rpy="0 0 0"/><geometry><box size="${tray_length} ${tray_width} ${tray_wall_thickness}"/></geometry><material name="RejectBin"><color rgba="0.75 0.35 0.1 1.0"/></material></visual>
+   <collision><origin xyz="0 0 ${-tray_height + tray_wall_thickness / 2}" rpy="0 0 0"/><geometry><box size="${tray_length} ${tray_width} ${tray_wall_thickness}"/></geometry></collision>
    <visual><origin xyz="0 ${tray_width / 2 - tray_wall_thickness / 2} ${-tray_height / 2}" rpy="0 0 0"/><geometry><box size="${tray_length} ${tray_wall_thickness} ${tray_height}"/></geometry></visual>
    <collision><origin xyz="0 ${tray_width / 2 - tray_wall_thickness / 2} ${-tray_height / 2}" rpy="0 0 0"/><geometry><box size="${tray_length} ${tray_wall_thickness} ${tray_height}"/></geometry></collision>
@@ -198,8 +214,8 @@
    <collision><origin xyz="${-tray_length / 2 + tray_wall_thickness / 2} 0 ${-tray_height / 2}" rpy="0 0 0"/><geometry><box size="${tray_wall_thickness} ${tray_width} ${tray_height}"/></geometry></collision>
  </link>
- <joint name="world_to_reject_bin" type="fixed">
-   <parent link="world"/>
+ <joint name="table_to_reject_bin" type="fixed">
+   <parent link="table_"/>
    <child link="reject_bin"/>
-   <origin xyz="${destination_area_x} 0.24 ${table_top_z + tray_wall_thickness}" rpy="0 0 0"/>
+   <origin xyz="${destination_area_x} 0.24 ${tray_height}" rpy="0 0 0"/>
  </joint>
  <!-- Pickup area: three items arranged in a reachable row on the tabletop (bottoms at table_top_z). -->
@@ -208,8 +224,8 @@
    <collision><geometry><box size="0.04 0.04 0.08"/></geometry></collision>
  </link>
- <joint name="world_to_item_red" type="fixed">
-   <parent link="world"/>
+ <joint name="table_to_item_red" type="fixed">
+   <parent link="table_"/>
    <child link="item_red"/>
-   <origin xyz="${pickup_area_x} ${pickup_area_y} ${table_top_z + item_red_height / 2}" rpy="0 0 0"/>
+   <origin xyz="${pickup_area_x} ${pickup_area_y} ${item_red_height / 2}" rpy="0 0 0"/>
  </joint>
  <link name="item_blue">
@@ -217,8 +233,8 @@
    <collision><geometry><cylinder length="0.06" radius="0.02"/></geometry></collision>
  </link>
- <joint name="world_to_item_blue" type="fixed">
-   <parent link="world"/>
+ <joint name="table_to_item_blue" type="fixed">
+   <parent link="table_"/>
    <child link="item_blue"/>
-   <origin xyz="${pickup_area_x + 0.08} ${pickup_area_y} ${table_top_z + item_blue_length / 2}" rpy="0 0 0"/>
+   <origin xyz="${pickup_area_x + 0.08} ${pickup_area_y} ${item_blue_length / 2}" rpy="0 0 0"/>
  </joint>
  <link name="item_green">
@@ -226,8 +242,8 @@
    <collision><geometry><sphere radius="0.025"/></geometry></collision>
  </link>
- <joint name="world_to_item_green" type="fixed">
-   <parent link="world"/>
+ <joint name="table_to_item_green" type="fixed">
+   <parent link="table_"/>
    <child link="item_green"/>
-   <origin xyz="${pickup_area_x + 0.16} ${pickup_area_y} ${table_top_z + item_green_radius}" rpy="0 0 0"/>
+   <origin xyz="${pickup_area_x + 0.16} ${pickup_area_y} ${item_green_radius}" rpy="0 0 0"/>
  </joint>
 </robot>

Commit message: Fix sorting scene pickup layout and table-relative validation

File: scenes/ur5_2f_sorting_test/urdf/scene.urdf.xacro (robot description, xacro)
@@ -19,6 +19,6 @@
  <xacro:property name="item_blue_length" value="0.06"/>
  <xacro:property name="item_green_radius" value="0.025"/>
- <xacro:property name="pickup_area_x" value="0.28"/>
- <xacro:property name="pickup_area_y" value="-0.12"/>
+ <xacro:property name="pickup_area_x" value="0.12"/>
+ <xacro:property name="pickup_area_y" value="0.00"/>
  <xacro:property name="destination_area_x" value="0.44"/>
  <xacro:property name="table_leg_size" value="0.07"/>
@@ -30,19 +30,19 @@
  <link name="table_">
    <visual>
-     <origin xyz="0 0 ${-(table_height - table_top_thickness) / 2}" rpy="0 0 0"/>
+     <origin xyz="0 0 ${-table_top_thickness - (table_height - table_top_thickness) / 2}" rpy="0 0 0"/>
      <geometry><box size="${table_length} ${table_width} ${table_height - table_top_thickness}"/></geometry>
      <material name="TableCabinet"><color rgba="0.46 0.33 0.24 1.0"/></material>
    </visual>
    <collision>
-     <origin xyz="0 0 ${-(table_height - table_top_thickness) / 2}" rpy="0 0 0"/>
+     <origin xyz="0 0 ${-table_top_thickness - (table_height - table_top_thickness) / 2}" rpy="0 0 0"/>
      <geometry><box size="${table_length} ${table_width} ${table_height - table_top_thickness}"/></geometry>
    </collision>
    <visual>
-     <origin xyz="0 0 ${table_top_thickness / 2}" rpy="0 0 0"/>
+     <origin xyz="0 0 ${-table_top_thickness / 2}" rpy="0 0 0"/>
      <geometry><box size="${table_length} ${table_width} ${table_top_thickness}"/></geometry>
      <material name="TableTop"><color rgba="0.55 0.40 0.28 1.0"/></material>
    </visual>
    <collision>
-     <origin xyz="0 0 ${table_top_thickness / 2}" rpy="0 0 0"/>
+     <origin xyz="0 0 ${-table_top_thickness / 2}" rpy="0 0 0"/>
      <geometry><box size="${table_length} ${table_width} ${table_top_thickness}"/></geometry>
    </collision>
@@ -119,10 +119,10 @@
  <link name="bin_a">
    <visual>
-     <origin xyz="0 0 ${-tray_wall_thickness / 2}" rpy="0 0 0"/>
+     <origin xyz="0 0 ${-tray_height + tray_wall_thickness / 2}" rpy="0 0 0"/>
      <geometry><box size="${tray_length} ${tray_width} ${tray_wall_thickness}"/></geometry>
      <material name="Blue"><color rgba="0.2 0.2 0.8 1.0"/></material>
    </visual>
    <collision>
-     <origin xyz="0 0 ${-tray_wall_thickness / 2}" rpy="0 0 0"/>
+     <origin xyz="0 0 ${-tray_height + tray_wall_thickness / 2}" rpy="0 0 0"/>
      <geometry><box size="${tray_length} ${tray_width} ${tray_wall_thickness}"/></geometry>
    </collision>
@@ -160,16 +160,16 @@
    </collision>
  </link>
- <joint name="world_to_bin_a" type="fixed">
-   <parent link="world"/>
+ <joint name="table_to_bin_a" type="fixed">
+   <parent link="table_"/>
    <child link="bin_a"/>
-   <origin xyz="${destination_area_x} -0.24 ${table_top_z + tray_wall_thickness}" rpy="0 0 0"/>
+   <origin xyz="${destination_area_x} -0.24 ${tray_height}" rpy="0 0 0"/>
  </joint>
  <link name="bin_b">
    <visual>
-     <origin xyz="0 0 ${-tray_wall_thickness / 2}" rpy="0 0 0"/>
+     <origin xyz="0 0 ${-tray_height + tray_wall_thickness / 2}" rpy="0 0 0"/>
      <geometry><box size="${tray_length} ${tray_width} ${tray_wall_thickness}"/></geometry>
      <material name="Green"><color rgba="0.2 0.8 0.2 1.0"/></material>
    </visual>
-   <collision><origin xyz="0 0 ${-tray_wall_thickness / 2}" rpy="0 0 0"/><geometry><box size="${tray_length} ${tray_width} ${tray_wall_thickness}"/></geometry></collision>
+   <collision><origin xyz="0 0 ${-tray_height + tray_wall_thickness / 2}" rpy="0 0 0"/><geometry><box size="${tray_length} ${tray_width} ${tray_wall_thickness}"/></geometry></collision>
    <visual><origin xyz="0 ${tray_width / 2 - tray_wall_thickness / 2} ${-tray_height / 2}" rpy="0 0 0"/><geometry><box size="${tray_length} ${tray_wall_thickness} ${tray_height}"/></geometry></visual>
    <collision><origin xyz="0 ${tray_width / 2 - tray_wall_thickness / 2} ${-tray_height / 2}" rpy="0 0 0"/><geometry><box size="${tray_length} ${tray_wall_thickness} ${tray_height}"/></geometry></collision>
@@ -181,12 +181,12 @@
    <collision><origin xyz="${-tray_length / 2 + tray_wall_thickness / 2} 0 ${-tray_height / 2}" rpy="0 0 0"/><geometry><box size="${tray_wall_thickness} ${tray_width} ${tray_height}"/></geometry></collision>
  </link>
- <joint name="world_to_bin_b" type="fixed">
-   <parent link="world"/>
+ <joint name="table_to_bin_b" type="fixed">
+   <parent link="table_"/>
    <child link="bin_b"/>
-   <origin xyz="${destination_area_x} 0.0 ${table_top_z + tray_wall_thickness}" rpy="0 0 0"/>
+   <origin xyz="${destination_area_x} 0.0 ${tray_height}" rpy="0 0 0"/>
  </joint>
  <link name="reject_bin">
-   <visual><origin xyz="0 0 ${-tray_wall_thickness / 2}" rpy="0 0 0"/><geometry><box size="${tray_length} ${tray_width} ${tray_wall_thickness}"/></geometry><material name="RejectBin"><color rgba="0.75 0.35 0.1 1.0"/></material></visual>
-   <collision><origin xyz="0 0 ${-tray_wall_thickness / 2}" rpy="0 0 0"/><geometry><box size="${tray_length} ${tray_width} ${tray_wall_thickness}"/></geometry></collision>
+   <visual><origin xyz="0 0 ${-tray_height + tray_wall_thickness / 2}" rpy="0 0 0"/><geometry><box size="${tray_length} ${tray_width} ${tray_wall_thickness}"/></geometry><material name="RejectBin"><color rgba="0.75 0.35 0.1 1.0"/></material></visual>
+   <collision><origin xyz="0 0 ${-tray_height + tray_wall_thickness / 2}" rpy="0 0 0"/><geometry><box size="${tray_length} ${tray_width} ${tray_wall_thickness}"/></geometry></collision>
    <visual><origin xyz="0 ${tray_width / 2 - tray_wall_thickness / 2} ${-tray_height / 2}" rpy="0 0 0"/><geometry><box size="${tray_length} ${tray_wall_thickness} ${tray_height}"/></geometry></visual>
    <collision><origin xyz="0 ${tray_width / 2 - tray_wall_thickness / 2} ${-tray_height / 2}" rpy="0 0 0"/><geometry><box size="${tray_length} ${tray_wall_thickness} ${tray_height}"/></geometry></collision>
@@ -198,8 +198,8 @@
    <collision><origin xyz="${-tray_length / 2 + tray_wall_thickness / 2} 0 ${-tray_height / 2}" rpy="0 0 0"/><geometry><box size="${tray_wall_thickness} ${tray_width} ${tray_height}"/></geometry></collision>
  </link>
- <joint name="world_to_reject_bin" type="fixed">
-   <parent link="world"/>
+ <joint name="table_to_reject_bin" type="fixed">
+   <parent link="table_"/>
    <child link="reject_bin"/>
-   <origin xyz="${destination_area_x} 0.24 ${table_top_z + tray_wall_thickness}" rpy="0 0 0"/>
+   <origin xyz="${destination_area_x} 0.24 ${tray_height}" rpy="0 0 0"/>
  </joint>
  <!-- Pickup area: three items arranged in a reachable row on the tabletop (bottoms at table_top_z). -->
@@ -208,8 +208,8 @@
    <collision><geometry><box size="0.04 0.04 0.08"/></geometry></collision>
  </link>
- <joint name="world_to_item_red" type="fixed">
-   <parent link="world"/>
+ <joint name="table_to_item_red" type="fixed">
+   <parent link="table_"/>
    <child link="item_red"/>
-   <origin xyz="${pickup_area_x} ${pickup_area_y} ${table_top_z + item_red_height / 2}" rpy="0 0 0"/>
+   <origin xyz="${pickup_area_x} ${pickup_area_y - 0.12} ${item_red_height / 2}" rpy="0 0 0"/>
  </joint>
  <link name="item_blue">
@@ -217,8 +217,8 @@
    <collision><geometry><cylinder length="0.06" radius="0.02"/></geometry></collision>
  </link>
- <joint name="world_to_item_blue" type="fixed">
-   <parent link="world"/>
+ <joint name="table_to_item_blue" type="fixed">
+   <parent link="table_"/>
    <child link="item_blue"/>
-   <origin xyz="${pickup_area_x + 0.08} ${pickup_area_y} ${table_top_z + item_blue_length / 2}" rpy="0 0 0"/>
+   <origin xyz="${pickup_area_x} ${pickup_area_y} ${item_blue_length / 2}" rpy="0 0 0"/>
  </joint>
  <link name="item_green">
@@ -226,8 +226,8 @@
    <collision><geometry><sphere radius="0.025"/></geometry></collision>
  </link>
- <joint name="world_to_item_green" type="fixed">
-   <parent link="world"/>
+ <joint name="table_to_item_green" type="fixed">
+   <parent link="table_"/>
    <child link="item_green"/>
-   <origin xyz="${pickup_area_x + 0.16} ${pickup_area_y} ${table_top_z + item_green_radius}" rpy="0 0 0"/>
+   <origin xyz="${pickup_area_x} ${pickup_area_y + 0.12} ${item_green_radius}" rpy="0 0 0"/>
  </joint>
 </robot>
