Commit message: Add workbench description package and modernize yaml loading

File: scenes/ur5_2f_test/urdf/scene.urdf.xacro (robot description, xacro)
@@ -17,11 +17,13 @@
 	<origin xyz="0 0 0" rpy="1.5707 -1.5707 0"/>
  </xacro:robotiq_85_gripper>
- <xacro:include filename="$(find table_description)/urdf/table.urdf.xacro"/>
- <xacro:table prefix="" parent="world">
-	<origin xyz="0 0 0" rpy="0 0 0"/>
- </xacro:table>
+ <xacro:include filename="$(find-pkg-share workbench_description)/urdf/workbench.urdf.xacro"/>
+ <joint name="workbench_base_joint" type="fixed">
+        <parent link="world" />
+        <child link="workbench_link" />
+        <origin xyz="0 0 0" rpy="0 0 0"/>
+ </joint>
  <xacro:include filename="$(find realsense2_description)/urdf/_d415.urdf.xacro"/>
  <xacro:arg name="use_nominal_extrinsics" default="true" />
- <xacro:sensor_d415 parent="table_" use_nominal_extrinsics="$(arg use_nominal_extrinsics)">
+ <xacro:sensor_d415 parent="workbench_link" use_nominal_extrinsics="$(arg use_nominal_extrinsics)">
     <origin xyz="-0.58 0.12 0.655" rpy="0 1.57079506 0"/>
  </xacro:sensor_d415>

File: scenes/ur5_3f_test/urdf/scene.urdf.xacro (robot description, xacro)
@@ -21,11 +21,13 @@
 	<origin xyz="0 0 0.0" rpy="1.5707 0 0"/>
  </xacro:robotiq-3f-gripper_articulated>
- <xacro:include filename="$(find table_description)/urdf/table.urdf.xacro"/>
- <xacro:table prefix="" parent="world">
-	<origin xyz="0 0 0" rpy="0 0 0"/>
- </xacro:table>
+ <xacro:include filename="$(find-pkg-share workbench_description)/urdf/workbench.urdf.xacro"/>
+ <joint name="workbench_base_joint" type="fixed">
+        <parent link="world" />
+        <child link="workbench_link" />
+        <origin xyz="0 0 0" rpy="0 0 0"/>
+ </joint>
  <xacro:include filename="$(find realsense2_description)/urdf/_d415.urdf.xacro"/>
 <xacro:arg name="use_nominal_extrinsics" default="true" />
-<xacro:sensor_d415 parent="table_" use_nominal_extrinsics="$(arg use_nominal_extrinsics)">
+<xacro:sensor_d415 parent="workbench_link" use_nominal_extrinsics="$(arg use_nominal_extrinsics)">
     <origin xyz="-0.58 0.225 0.65" rpy="3.14159 1.57079506 0"/>
 </xacro:sensor_d415>

File: scenes/ur5_airpick4_test/urdf/scene.urdf.xacro (robot description, xacro)
@@ -13,8 +13,10 @@
  <xacro:arg name="initial_positions_file" default="$(find ur5_moveit_config)/config/initial_positions.yaml" />
  <xacro:ur5_ros2_control name="UR5FakeSystem" initial_positions_file="$(arg initial_positions_file)"/>
- <xacro:include filename="$(find table_description)/urdf/table.urdf.xacro"/>
- <xacro:table prefix="" parent="world">
-	<origin xyz="0 0 0" rpy="0 0 0"/>
- </xacro:table>
+ <xacro:include filename="$(find-pkg-share workbench_description)/urdf/workbench.urdf.xacro"/>
+ <joint name="workbench_base_joint" type="fixed">
+        <parent link="world" />
+        <child link="workbench_link" />
+        <origin xyz="0 0 0" rpy="0 0 0"/>
+ </joint>
   <!--xacro:include filename="$(find realsense2_description)/urdf/_d415.urdf.xacro"/>
  <xacro:arg name="use_nominal_extrinsics" default="true" />
@@ -25,5 +27,5 @@
  <xacro:include filename="$(find realsense2_description)/urdf/_d415.urdf.xacro"/>
  <xacro:arg name="use_nominal_extrinsics" default="true" />
- <xacro:sensor_d415 parent="table_" use_nominal_extrinsics="$(arg use_nominal_extrinsics)">
+ <xacro:sensor_d415 parent="workbench_link" use_nominal_extrinsics="$(arg use_nominal_extrinsics)">
 	<origin xyz="-0.58 0.225 0.65" rpy="3.14159 1.57079506 0"/>
  </xacro:sensor_d415>

Commit message: Align ur5_2f_test scene contract

File: scenes/ur5_2f_test/urdf/scene.urdf.xacro (robot description, xacro)
@@ -4,11 +4,17 @@
  <xacro:arg name="name" default="$(arg ur_type)"/>
  <xacro:arg name="tf_prefix" default=""/>
+ <xacro:arg name="world_frame" default="world"/>
+ <xacro:arg name="tool_mount_link" default="tool0"/>
+ <xacro:arg name="gripper_profile" default="robotiq_85_gripper"/>
+ <xacro:arg name="grasp_frame" default="ee_palm"/>
  <xacro:arg name="use_fake_hardware" default="true"/>
- <link name="world"/>
+ <!-- Contract: world_frame is the scene/world frame; UR creates base_link as the robot base. -->
+ <!-- Contract: tool_mount_link is tool0; gripper_profile is robotiq_85_gripper; grasp_frame is ee_palm. -->
+ <link name="$(arg world_frame)"/>
 <xacro:include filename="$(find ur_description)/urdf/ur_macro.xacro"/>
 <xacro:ur_robot
   name="$(arg name)"
   tf_prefix="$(arg tf_prefix)"
-  parent="world"
+  parent="$(arg world_frame)"
   safety_limits="true"
   joint_limits_parameters_file="$(find ur_description)/config/$(arg ur_type)/joint_limits.yaml"
@@ -20,5 +26,5 @@
 </xacro:ur_robot>
  <xacro:include filename="$(find robotiq_85_description)/urdf/robotiq_85_gripper.urdf.xacro"/>
- <xacro:robotiq_85_gripper prefix="" parent="tool0">
+ <xacro:robotiq_85_gripper prefix="" parent="$(arg tool_mount_link)">
 	<origin xyz="0 0 0" rpy="1.5707 -1.5707 0"/>
  </xacro:robotiq_85_gripper>
@@ -40,5 +46,5 @@
  </xacro:if>
  <xacro:include filename="$(find workbench_description)/urdf/table.urdf.xacro"/>
- <xacro:table prefix="" parent="world">
+ <xacro:table prefix="" parent="$(arg world_frame)">
 	<origin xyz="0 0 0" rpy="0 0 0"/>
  </xacro:table>
@@ -55,8 +61,8 @@
     <origin xyz="0 0 0" rpy="1.57079506 0 1.57079506"/>
  </joint>
- <link name="ee_palm" />
- <joint name="base_to_palm" type="fixed">
-    <parent link="tool0"/>
-    <child link="ee_palm"/>
+ <link name="$(arg grasp_frame)" />
+ <joint name="tool0_to_grasp_frame" type="fixed">
+    <parent link="$(arg tool_mount_link)"/>
+    <child link="$(arg grasp_frame)"/>
     <origin xyz="0 0 0.14" rpy="0 0 0"/>
  </joint>
