Commit message: Load canonical layout poses in ur5 RViz launch

File: scenes/ur5_2f_test/urdf/scene.urdf.xacro (robot description, xacro)
@@ -9,4 +9,8 @@
  <xacro:arg name="grasp_frame" default="ee_palm"/>
  <xacro:arg name="use_fake_hardware" default="true"/>
+ <xacro:arg name="table_world_xyz"/>
+ <xacro:arg name="table_world_rpy"/>
+ <xacro:arg name="camera_world_xyz"/>
+ <xacro:arg name="camera_world_rpy"/>
  <!-- Contract: world_frame is the scene/world frame; UR creates base_link as the robot base. -->
  <!-- Contract: tool_mount_link is tool0; gripper_profile is robotiq_85_gripper; grasp_frame is ee_palm. -->
@@ -47,10 +51,10 @@
  <xacro:include filename="$(find workbench_description)/urdf/table.urdf.xacro"/>
  <xacro:table prefix="" parent="$(arg world_frame)">
-	<origin xyz="0 0 0" rpy="0 0 0"/>
+	<origin xyz="$(arg table_world_xyz)" rpy="$(arg table_world_rpy)"/>
  </xacro:table>
  <xacro:include filename="$(find realsense2_description)/urdf/_d435i.urdf.xacro"/>
  <xacro:arg name="use_nominal_extrinsics" default="true" />
- <xacro:sensor_d435i parent="table_" use_nominal_extrinsics="$(arg use_nominal_extrinsics)">
-    <origin xyz="-0.58 0.12 0.655" rpy="0 1.57079506 0"/>
+ <xacro:sensor_d435i parent="$(arg world_frame)" use_nominal_extrinsics="$(arg use_nominal_extrinsics)">
+    <origin xyz="$(arg camera_world_xyz)" rpy="$(arg camera_world_rpy)"/>
  </xacro:sensor_d435i>
  <link name="camera_frame" />

Commit message: Fix ur5_2f_test planning start collision

File: scenes/ur5_2f_test/urdf/scene.urdf.xacro (robot description, xacro)
@@ -27,5 +27,6 @@
   visual_parameters_file="$(find ur_description)/config/$(arg ur_type)/visual_parameters.yaml"
   use_fake_hardware="$(arg use_fake_hardware)">
-  <origin xyz="0 0 0" rpy="0 0 0"/>
+  <!-- The reviewed support-surface proxy has its top at world z=0.10 m. -->
+  <origin xyz="0 0 0.10" rpy="0 0 0"/>
 </xacro:ur_robot>
  <xacro:include filename="$(find robotiq_85_description)/urdf/robotiq_85_gripper.urdf.xacro"/>

Commit message: R1.3: drive UR5 fake-hardware start from canonical Robot Home

File: scenes/ur5_2f_test/urdf/scene.urdf.xacro (robot description, xacro)
@@ -15,4 +15,9 @@
  <xacro:arg name="camera_world_xyz" default=""/>
  <xacro:arg name="camera_world_rpy" default=""/>
+ <xacro:arg name="environment_file" default="$(find ur5_2f_test)/environment.yaml"/>
+ <!-- The canonical scene-local Robot Home is authored in environment.yaml. -->
+ <xacro:property name="environment_file" default="$(arg environment_file)"/>
+ <xacro:property name="workcell_environment" value="${xacro.load_yaml(environment_file)}"/>
+ <xacro:property name="workcell_home_joint_state" value="${workcell_environment['robot']['home_joint_state']['joints']}"/>
  <!-- Contract: world_frame is the scene/world frame; UR creates base_link as the robot base. -->
  <!-- Contract: tool_mount_link is tool0; gripper_profile is robotiq_85_gripper; grasp_frame is ee_palm. -->
@@ -28,5 +33,6 @@
   physical_parameters_file="$(find ur_description)/config/$(arg ur_type)/physical_parameters.yaml"
   visual_parameters_file="$(find ur_description)/config/$(arg ur_type)/visual_parameters.yaml"
-  use_fake_hardware="$(arg use_fake_hardware)">
+  use_fake_hardware="$(arg use_fake_hardware)"
+  initial_positions="${workcell_home_joint_state}">
   <!-- Authored robot mounting pose; the mounting plate and workbench are
        separate PlanningScene objects generated from the saved environment. -->
