Commit message: Complete UR5 Robotiq industrial workcell handoff

File: scenes/ur5_2f_test/urdf/arm_hand.srdf.xacro (robot description, xacro)
@@ -5,12 +5,10 @@
   <xacro:ur5/>
   <xacro:robotiq_85_gripper/>
-  <disable_collisions link1="gripper_base_link" link2="base_link" reason="Never" />
-  <disable_collisions link1="gripper_base_link" link2="shoulder_link" reason="Never" />
-  <disable_collisions link1="gripper_base_link" link2="upper_arm_link" reason="Never" />
-  <disable_collisions link1="gripper_base_link" link2="forearm_link" reason="Never" />
-  <disable_collisions link1="gripper_base_link" link2="wrist_1_link" reason="Never" />
-  <disable_collisions link1="gripper_base_link" link2="wrist_2_link" reason="Never" />
-  <disable_collisions link1="gripper_base_link" link2="wrist_3_link" reason="Never" />
+  <!-- Only the rigid mounting interface is exempted here.  The gripper
+       profile supplies its own adjacent-link pairs; broad exemptions against
+       the arm would hide a real self-collision. -->
   <disable_collisions link1="gripper_base_link" link2="tool0" reason="Never" />
-  <disable_collisions link1="gripper_base_link" link2="base" reason="Never" />
+  <!-- Explicit rigid adapter contact; this is the single mount exemption and
+       does not broaden the arm's self-collision matrix. -->
+  <disable_collisions link1="gripper_base_link" link2="wrist_3_link" reason="Adjacent" />
 </robot>

File: scenes/ur5_2f_test/urdf/scene.urdf.xacro (robot description, xacro)
@@ -9,4 +9,6 @@
  <xacro:arg name="grasp_frame" default="ee_palm"/>
  <xacro:arg name="use_fake_hardware" default="true"/>
+ <xacro:arg name="robot_world_xyz" default="0 0 0.0135"/>
+ <xacro:arg name="robot_world_rpy" default="0 0 0"/>
  <xacro:arg name="table_world_xyz" default=""/>
  <xacro:arg name="table_world_rpy" default=""/>
@@ -27,6 +29,7 @@
   visual_parameters_file="$(find ur_description)/config/$(arg ur_type)/visual_parameters.yaml"
   use_fake_hardware="$(arg use_fake_hardware)">
-  <!-- The reviewed support-surface proxy has its top at world z=0.10 m. -->
-  <origin xyz="0 0 0.10" rpy="0 0 0"/>
+  <!-- Authored robot mounting pose; the mounting plate and workbench are
+       separate PlanningScene objects generated from the saved environment. -->
+  <origin xyz="$(arg robot_world_xyz)" rpy="$(arg robot_world_rpy)"/>
 </xacro:ur_robot>
  <xacro:include filename="$(find robotiq_85_description)/urdf/robotiq_85_gripper.urdf.xacro"/>
@@ -50,8 +53,7 @@
    </ros2_control>
  </xacro:if>
- <xacro:include filename="$(find workbench_description)/urdf/table.urdf.xacro"/>
- <xacro:table prefix="" parent="$(arg world_frame)">
-	<origin xyz="$(arg table_world_xyz)" rpy="$(arg table_world_rpy)"/>
- </xacro:table>
+ <!-- The authored table is applied once by the MoveIt collision manifest.
+      Keeping a second URDF table here would create duplicate geometry and a
+      false table-vs-table contact in state validity checks. -->
  <xacro:include filename="$(find realsense2_description)/urdf/_d435i.urdf.xacro"/>
  <xacro:arg name="use_nominal_extrinsics" default="true" />
